Commit message: testtt

File: descriptions/stewart_little_magnet/robot.urdf (robot description, URDF)
Before this commit: robot robot, 39 links, 38 joints
Links:
- link platform: mass 0.0270567 -> 0.207267
Joints:
- joint 1: child right_arm -> left_arm; origin xyz=-0.00838143 -0.0495171 0.0434238 rpy=-1.86732 -0.377171 -0.411546 -> xyz=-0.0386923 -0.0320171 0.0434238 rpy=-1.86732 0.377171 -0.635652
- joint 2: child left_arm -> right_arm; origin xyz=-0.0386923 -0.0320171 0.0434238 rpy=-1.86732 0.377171 -0.635652 -> xyz=-0.00838143 -0.0495171 0.0434238 rpy=-1.86732 -0.377171 -0.411546
- joint 3: origin xyz=-0.00838053 0.0495175 0.0434241 rpy=-1.86731 0.37714 -2.73004 -> xyz=0.0470734 -0.017499 0.0434252 rpy=-1.86732 0.377203 1.45873
- joint 4: origin xyz=-0.0386913 0.0320172 0.0434252 rpy=-1.86732 -0.377203 -2.50593 -> xyz=0.0470737 0.017501 0.0434241 rpy=-1.86731 -0.37714 1.68284
- joint 5: origin xyz=0.0470734 -0.017499 0.0434252 rpy=-1.86732 0.377203 1.45873 -> xyz=-0.00838053 0.0495175 0.0434241 rpy=-1.86731 0.37714 -2.73004
- joint 6: origin xyz=0.0470737 0.017501 0.0434241 rpy=-1.86731 -0.37714 1.68284 -> xyz=-0.0386913 0.0320172 0.0434252 rpy=-1.86732 -0.377203 -2.50593
- joint closing_1_2_frame: parent 10mm_ball_3 -> 10mm_ball_5
- joint closing_4_1_frame: parent 10mm_ball_4 -> 10mm_ball_2
- joint closing_5_2_frame: parent 10mm_ball_5 -> 10mm_ball_3
- joint passive_2_x: parent right_arm_2 -> right_arm_3
- joint passive_2_z: child 10mm_ball_3 -> 10mm_ball_5
- joint passive_3_x: parent left_arm_2 -> left_arm_3
- joint passive_3_z: child 10mm_ball_2 -> 10mm_ball_4
- joint passive_4_x: parent right_arm_3 -> right_arm_2
- joint passive_4_z: child 10mm_ball_5 -> 10mm_ball_3
- joint passive_5_x: parent left_arm_3 -> left_arm_2
- joint passive_5_z: child 10mm_ball_4 -> 10mm_ball_2
- joint passive_7_x: parent 10mm_ball_2 -> 10mm_ball_4

Commit message: update model to use antennas

File: descriptions/stewart_little_magnet/robot.urdf (robot description, URDF)
Before this commit: robot robot, 39 links, 38 joints
Links:
- added link pp00672_antenna_mic_a1, mass 0.0202419; collision mesh filename=package://assets/pp00672_antenna_mic_a1.stl; collision mesh filename=package://assets/pp00673_antenna_sphere_a1.stl
- added link pp00672_antenna_mic_a1_2, mass 0.0202419; collision mesh filename=package://assets/pp00672_antenna_mic_a1.stl; collision mesh filename=package://assets/pp00673_antenna_sphere_a1.stl
- link platform: mass 0.207267 -> 0.363548; geometry collision mesh filename=package://assets/magnet.stl; collision mesh filename=package://assets/magnet.stl
Joints:
- added joint left_antenna: type revolute, parent platform, child pp00672_antenna_mic_a1, origin xyz=0.035159 -0.0622228 0.0749453 rpy=2.08187 1.01498 -1.71429, axis 0 0 1, limit lower=-3.141592653589793 upper=3.141592653589793 effort=10 velocity=10
- added joint right_antenna: type revolute, parent platform, child pp00672_antenna_mic_a1_2, origin xyz=-0.0202961 0.0200517 0.122439 rpy=2.64924 -0.230354 -0.605094, axis 0 0 1, limit lower=-3.141592653589793 upper=3.141592653589793 effort=10 velocity=10
- joint closing_1_2_frame: origin xyz=4.71845e-16 -1.04083e-17 0.0996012 rpy=1.01844e-14 8.6843e-16 5.72444e-16 -> xyz=5.27356e-16 3.46945e-18 0.0996012 rpy=1.01567e-14 8.6843e-16 5.16933e-16
- joint closing_3_2_frame: origin xyz=1.08941e-15 0 0.0996012 rpy=4.75183e-15 4.22036e-16 -1.23095e-16 -> xyz=1.07553e-15 1.38778e-17 0.0996012 rpy=4.68876e-15 3.84954e-16 -1.1657e-16
- joint closing_4_1_frame: origin xyz=-4.23273e-16 1.38778e-17 0.0996012 rpy=-3.14159 -7.93145e-16 -3.14159 -> xyz=-4.3715e-16 2.08167e-17 0.0996012 rpy=-3.14159 -8.209e-16 -3.14159
- joint closing_5_1_frame: origin xyz=-0.023093 0 -0.000220061 rpy=-3.58553e-15 -0.0190581 7.56579e-17 -> xyz=-0.023093 2.77556e-17 -0.000220061 rpy=-3.5922e-15 -0.0190581 -1.36686e-16
- joint closing_5_2_frame: origin xyz=-9.22873e-16 9.71445e-17 0.0996012 rpy=2.72084e-14 -1.09948e-15 1.5708 -> xyz=-9.64506e-16 5.55112e-17 0.0996012 rpy=2.6558e-14 -9.92746e-16 1.5708
- joint passive_1_x: origin xyz=-0.038 6.93889e-17 0.00384958 rpy=-1.5708 -4.30224e-17 3.14159 -> xyz=-0.038 6.245e-17 0.00384958 rpy=-1.5708 1.10155e-16 3.14159
- joint passive_1_y: origin xyz=-1.38778e-17 -6.93889e-18 0 rpy=4.02934e-18 -1.59424e-17 6.78641e-17 -> xyz=1.38778e-17 -6.93889e-18 -3.46945e-18 rpy=-1.91261e-17 3.04674e-17 5.37636e-17
- joint passive_1_z: origin xyz=-1.38778e-17 -6.93889e-18 0 rpy=4.02934e-18 -1.59424e-17 6.78641e-17 -> xyz=1.38778e-17 -6.93889e-18 -3.46945e-18 rpy=-1.91261e-17 3.04674e-17 5.37636e-17
- joint passive_2_x: origin xyz=0.038 -7.63278e-17 0.00384958 rpy=1.67139 1.0009 0.0518494 -> xyz=0.038 -3.19189e-16 0.00384958 rpy=1.67139 1.0009 0.0518494
- joint passive_2_y: origin xyz=-1.38778e-17 -3.46945e-18 0 rpy=2.60495e-17 1.50798e-17 3.3994e-18 -> xyz=1.38778e-17 3.46945e-18 0 rpy=2.2995e-17 -4.04313e-17 -1.04784e-17
- joint passive_2_z: origin xyz=-1.38778e-17 -3.46945e-18 0 rpy=2.60495e-17 1.50798e-17 3.3994e-18 -> xyz=1.38778e-17 3.46945e-18 0 rpy=2.2995e-17 -4.04313e-17 -1.04784e-17
- joint passive_3_x: origin xyz=-0.038 -1.35308e-16 0.00384958 rpy=1.68969 1.09636 0.138717 -> xyz=-0.038 -1.56125e-16 0.00384958 rpy=1.68969 1.09636 0.138717
- joint passive_3_y: origin xyz=-3.46945e-18 0 0 rpy=6.75164e-18 1.08153e-18 -3.57996e-17 -> xyz=-6.93889e-18 0 0 rpy=8.6686e-17 -5.53998e-17 3.69236e-17
- joint passive_3_z: origin xyz=-3.46945e-18 0 0 rpy=6.75164e-18 1.08153e-18 -3.57996e-17 -> xyz=-6.93889e-18 0 0 rpy=8.6686e-17 -5.53998e-17 3.69236e-17
- joint passive_4_x: origin xyz=0.038 -6.245e-17 0.00384958 rpy=1.63153 -0.467373 -0.0602377 -> xyz=0.038 -1.14492e-16 0.00384958 rpy=1.63153 -0.467373 -0.0602377
- joint passive_4_y: origin xyz=0 0 6.93889e-18 rpy=-6.87265e-18 -4.82997e-17 7.8678e-17 -> xyz=0 -1.38778e-17 0 rpy=-5.80953e-17 -3.20322e-17 6.66802e-17
- joint passive_4_z: origin xyz=0 0 6.93889e-18 rpy=-6.87265e-18 -4.82997e-17 7.8678e-17 -> xyz=0 -1.38778e-17 0 rpy=-5.80953e-17 -3.20322e-17 6.66802e-17
- joint passive_5_x: origin xyz=-0.038 -6.93889e-18 0.00384958 rpy=1.94647 -1.42258 -0.338994 -> xyz=-0.038 -3.46945e-18 0.00384958 rpy=1.94647 -1.42258 -0.338994
- joint passive_5_y: origin xyz=0 6.93889e-18 0 rpy=-5.28992e-17 -2.05212e-17 -2.0417e-17 -> xyz=-6.93889e-18 6.93889e-18 0 rpy=4.59049e-17 -2.05212e-17 -1.09212e-17
- joint passive_5_z: origin xyz=0 6.93889e-18 0 rpy=-5.28992e-17 -2.05212e-17 -2.0417e-17 -> xyz=-6.93889e-18 6.93889e-18 0 rpy=4.59049e-17 -2.05212e-17 -1.09212e-17
- joint passive_6_x: origin xyz=0.038 2.42861e-17 0.00384958 rpy=-1.63195 0.485977 3.08012 -> xyz=0.038 4.51028e-17 0.00384958 rpy=-1.63195 0.485977 3.08012
- joint passive_6_y: origin xyz=0 0 0 rpy=4.33205e-17 1.67833e-17 -1.5514e-18 -> xyz=0 0 -3.46945e-18 rpy=2.96551e-17 -2.02993e-17 4.97353e-18
- joint passive_6_z: origin xyz=0 0 0 rpy=4.33205e-17 1.67833e-17 -1.5514e-18 -> xyz=0 0 -3.46945e-18 rpy=2.96551e-17 -2.02993e-17 4.97353e-18
- joint passive_7_x: origin xyz=5.55112e-17 2.77556e-17 0.0996012 rpy=-0.0563544 -0.0277816 0.113755 -> xyz=7.63278e-17 4.16334e-17 0.0996012 rpy=-0.0563544 -0.0277816 0.113755
- joint passive_7_y: origin xyz=1.38778e-17 -1.38778e-17 -1.38778e-17 rpy=-6.95244e-18 1.4546e-17 -6.26056e-17 -> xyz=3.46945e-18 -1.38778e-17 -1.38778e-17 rpy=-1.3621e-17 -3.08255e-17 -6.96528e-17
- joint passive_7_z: origin xyz=1.38778e-17 -1.38778e-17 -1.38778e-17 rpy=-6.95244e-18 1.4546e-17 -6.26056e-17 -> xyz=3.46945e-18 -1.38778e-17 -1.38778e-17 rpy=-1.3621e-17 -3.08255e-17 -6.96528e-17
