Commit message: reachy home v1

File: descriptions/reachy_home_v1/robot.urdf (robot description, URDF)
Before this commit: robot reachy_home, 41 links, 40 joints
Links:
- added link head, mass 1e-9
- link plateform: geometry collision mesh filename=package://assets/ball.stl; collision mesh filename=package://assets/ball.stl
Joints:
- added joint head_frame: type fixed, parent plateform, child head, origin xyz=0.00367542 0.0183217 -0.0274783 rpy=-1.74312 -0.143141 -1.99997, axis 0 0 0

Commit message: head and hand tracking utilities and demos

File: descriptions/reachy_home_v1/robot.urdf (robot description, URDF)
Before this commit: robot robot, 42 links, 41 joints
Joints:
- joint 1: limit lower=-3.141592653589793 upper=3.141592653589793 effort=10 velocity=10 -> lower=-1.39626 upper=1.39626 effort=10 velocity=10
- joint 2: limit lower=-3.141592653589793 upper=3.141592653589793 effort=10 velocity=10 -> lower=-1.39626 upper=1.39626 effort=10 velocity=10; origin xyz=0.0416206 0.012144 -0.044785 rpy=-1.5708 8.01479e-15 -1.0472 -> xyz=0.0416206 0.012144 -0.044785 rpy=-1.5708 1.45885e-14 -1.0472
- joint 3: limit lower=-3.141592653589793 upper=3.141592653589793 effort=10 velocity=10 -> lower=-1.39626 upper=1.39626 effort=10 velocity=10
- joint 4: limit lower=-3.141592653589793 upper=3.141592653589793 effort=10 velocity=10 -> lower=-1.39626 upper=1.39626 effort=10 velocity=10; origin xyz=-0.0102067 -0.0421165 -0.044785 rpy=-1.5708 5.55112e-17 -3.14159 -> xyz=-0.0102067 -0.0421165 -0.044785 rpy=-1.5708 4.43797e-15 -3.14159
- joint 5: limit lower=-3.141592653589793 upper=3.141592653589793 effort=10 velocity=10 -> lower=-1.39626 upper=1.39626 effort=10 velocity=10; origin xyz=-0.041534 0.012144 -0.044785 rpy=1.5708 -9.91031e-16 -2.0944 -> xyz=-0.041534 0.012144 -0.044785 rpy=1.5708 -6.46911e-15 -2.0944
- joint 6: limit lower=-3.141592653589793 upper=3.141592653589793 effort=10 velocity=10 -> lower=-1.39626 upper=1.39626 effort=10 velocity=10; origin xyz=-0.031284 0.0298975 -0.044785 rpy=-1.5708 -1.10323e-14 1.0472 -> xyz=-0.031284 0.0298975 -0.044785 rpy=-1.5708 -1.65104e-14 1.0472
- joint all_yaw: limit lower=-3.141592653589793 upper=3.141592653589793 effort=10 velocity=10 -> lower=-2.96706 upper=2.96706 effort=10 velocity=10
- joint closing_3_1_frame: origin xyz=-0.0900003 0 -1.11022e-16 rpy=-1.11647e-16 5.1013e-17 3.14159 -> xyz=-0.0900003 -1.38778e-17 -9.71445e-17 rpy=-1.09454e-16 6.55503e-17 3.14159
- joint closing_5_1_frame: origin xyz=-0.0900003 -6.93889e-18 1.70697e-15 rpy=-3.97878e-14 -2.23854e-14 -3.14159 -> xyz=-0.0900003 6.93889e-18 1.72085e-15 rpy=-3.97467e-14 -2.23603e-14 -3.14159
- joint passive_2_x: origin xyz=0.038 3.33067e-16 -0.00768 rpy=-0.186454 -0.0202587 -1.08831 -> xyz=0.038 8.32667e-17 -0.00768 rpy=-0.186454 -0.0202587 -1.08831
- joint passive_3_x: origin xyz=0.038 4.16334e-17 -0.00768 rpy=2.99943 -0.0202587 1.08831 -> xyz=0.038 -1.38778e-17 -0.00768 rpy=2.99943 -0.0202587 1.08831
- joint passive_3_y: origin xyz=-6.93889e-18 1.38778e-17 0 rpy=1.71657e-17 2.88559e-18 1.79253e-17 -> xyz=6.93889e-18 0 -3.46945e-18 rpy=1.84422e-17 -4.71284e-18 1.5244e-17
- joint passive_3_z: origin xyz=-6.93889e-18 1.38778e-17 0 rpy=1.71657e-17 2.88559e-18 1.79253e-17 -> xyz=6.93889e-18 0 -3.46945e-18 rpy=1.84422e-17 -4.71284e-18 1.5244e-17
- joint passive_4_x: origin xyz=0.038 -1.38778e-17 -0.00768 rpy=-2.75098 -0.0202587 -1.08831 -> xyz=0.038 -1.38778e-16 -0.00768 rpy=-2.75098 -0.0202587 -1.08831
- joint passive_5_y: origin xyz=6.93889e-18 6.93889e-18 0 rpy=-1.12808e-17 -1.80474e-17 -1.19975e-17 -> xyz=0 1.38778e-17 0 rpy=-3.59448e-17 -1.53626e-17 -3.22246e-17
- joint passive_5_z: origin xyz=6.93889e-18 6.93889e-18 0 rpy=-1.12808e-17 -1.80474e-17 -1.19975e-17 -> xyz=0 1.38778e-17 0 rpy=-3.59448e-17 -1.53626e-17 -3.22246e-17
- joint passive_6_x: origin xyz=0.038 9.71445e-17 -0.00768 rpy=-2.72876 -0.0202587 -1.08831 -> xyz=0.038 2.77556e-17 -0.00768 rpy=-2.72876 -0.0202587 -1.08831
- joint passive_6_y: origin xyz=-6.93889e-18 0 -1.84314e-18 rpy=-9.80843e-18 9.56019e-19 -2.78433e-17 -> xyz=-1.38778e-17 1.38778e-17 1.95156e-18 rpy=-5.18698e-17 -1.9094e-18 4.12252e-17
- joint passive_6_z: origin xyz=-6.93889e-18 0 -1.84314e-18 rpy=-9.80843e-18 9.56019e-19 -2.78433e-17 -> xyz=-1.38778e-17 1.38778e-17 1.95156e-18 rpy=-5.18698e-17 -1.9094e-18 4.12252e-17
- joint passive_7_x: origin xyz=-0.0900003 1.80411e-16 -7.58942e-18 rpy=3.14159 -3.24387e-17 3.14159 -> xyz=-0.0900003 2.22045e-16 -1.31188e-17 rpy=3.14159 -5.73288e-17 3.14159
- joint passive_7_y: origin xyz=0 1.38778e-17 -2.92735e-18 rpy=1.21162e-17 1.19364e-17 3.40244e-17 -> xyz=0 -1.38778e-17 -3.03577e-18 rpy=4.31179e-18 4.6347e-17 -7.78613e-17
- joint passive_7_z: origin xyz=0 1.38778e-17 -2.92735e-18 rpy=1.21162e-17 1.19364e-17 3.40244e-17 -> xyz=0 -1.38778e-17 -3.03577e-18 rpy=4.31179e-18 4.6347e-17 -7.78613e-17
