Commit message: fixed, we didn't step the kinematics solver enough

File: descriptions/reachy_mini/urdf/robot.urdf (robot description, URDF)
Before this commit: robot robot, 42 links, 41 joints
Joints:
- joint 1: limit lower=-1.39626 upper=1.39626 effort=10 velocity=10 -> lower=-1.39626 upper=1.39626 effort=10 velocity=8
- joint 2: limit lower=-1.39626 upper=1.39626 effort=10 velocity=10 -> lower=-1.39626 upper=1.39626 effort=10 velocity=8
- joint 3: limit lower=-1.39626 upper=1.39626 effort=10 velocity=10 -> lower=-1.39626 upper=1.39626 effort=10 velocity=8
- joint 4: limit lower=-1.39626 upper=1.39626 effort=10 velocity=10 -> lower=-1.39626 upper=1.39626 effort=10 velocity=8
- joint 5: limit lower=-1.39626 upper=1.39626 effort=10 velocity=10 -> lower=-1.39626 upper=1.39626 effort=10 velocity=8
- joint 6: limit lower=-1.39626 upper=1.39626 effort=10 velocity=10 -> lower=-1.39626 upper=1.39626 effort=10 velocity=8
- joint all_yaw: limit lower=-2.96706 upper=2.96706 effort=10 velocity=10 -> lower=-2.96706 upper=2.96706 effort=10 velocity=8
- joint left_antenna: limit lower=-3.141592653589793 upper=3.141592653589793 effort=10 velocity=10 -> lower=-3.141592653589793 upper=3.141592653589793 effort=10 velocity=8
- joint right_antenna: limit lower=-3.141592653589793 upper=3.141592653589793 effort=10 velocity=10 -> lower=-3.141592653589793 upper=3.141592653589793 effort=10 velocity=8

Commit message: bump onshape-to-robot version to 1.7.5, this version fixes a bug that didn't preserve the joint properties for ball_to_euler generated joints

File: descriptions/reachy_mini/urdf/robot.urdf (robot description, URDF)
Before this commit: robot robot, 42 links, 41 joints
Joints:
- joint passive_1_x: limit lower=-3.141592653589793 upper=3.141592653589793 effort=10 velocity=10 -> lower=-3.141592653589793 upper=3.141592653589793 effort=10 velocity=1e+08
- joint passive_1_y: limit lower=-3.141592653589793 upper=3.141592653589793 effort=10 velocity=10 -> lower=-3.141592653589793 upper=3.141592653589793 effort=10 velocity=1e+08
- joint passive_1_z: limit lower=-3.141592653589793 upper=3.141592653589793 effort=10 velocity=10 -> lower=-3.141592653589793 upper=3.141592653589793 effort=10 velocity=1e+08
- joint passive_2_x: limit lower=-3.141592653589793 upper=3.141592653589793 effort=10 velocity=10 -> lower=-3.141592653589793 upper=3.141592653589793 effort=10 velocity=1e+08
- joint passive_2_y: limit lower=-3.141592653589793 upper=3.141592653589793 effort=10 velocity=10 -> lower=-3.141592653589793 upper=3.141592653589793 effort=10 velocity=1e+08
- joint passive_2_z: limit lower=-3.141592653589793 upper=3.141592653589793 effort=10 velocity=10 -> lower=-3.141592653589793 upper=3.141592653589793 effort=10 velocity=1e+08
- joint passive_3_x: limit lower=-3.141592653589793 upper=3.141592653589793 effort=10 velocity=10 -> lower=-3.141592653589793 upper=3.141592653589793 effort=10 velocity=1e+08
- joint passive_3_y: limit lower=-3.141592653589793 upper=3.141592653589793 effort=10 velocity=10 -> lower=-3.141592653589793 upper=3.141592653589793 effort=10 velocity=1e+08
- joint passive_3_z: limit lower=-3.141592653589793 upper=3.141592653589793 effort=10 velocity=10 -> lower=-3.141592653589793 upper=3.141592653589793 effort=10 velocity=1e+08
- joint passive_4_x: limit lower=-3.141592653589793 upper=3.141592653589793 effort=10 velocity=10 -> lower=-3.141592653589793 upper=3.141592653589793 effort=10 velocity=1e+08
- joint passive_4_y: limit lower=-3.141592653589793 upper=3.141592653589793 effort=10 velocity=10 -> lower=-3.141592653589793 upper=3.141592653589793 effort=10 velocity=1e+08
- joint passive_4_z: limit lower=-3.141592653589793 upper=3.141592653589793 effort=10 velocity=10 -> lower=-3.141592653589793 upper=3.141592653589793 effort=10 velocity=1e+08
- joint passive_5_x: limit lower=-3.141592653589793 upper=3.141592653589793 effort=10 velocity=10 -> lower=-3.141592653589793 upper=3.141592653589793 effort=10 velocity=1e+08
- joint passive_5_y: limit lower=-3.141592653589793 upper=3.141592653589793 effort=10 velocity=10 -> lower=-3.141592653589793 upper=3.141592653589793 effort=10 velocity=1e+08
- joint passive_5_z: limit lower=-3.141592653589793 upper=3.141592653589793 effort=10 velocity=10 -> lower=-3.141592653589793 upper=3.141592653589793 effort=10 velocity=1e+08
- joint passive_6_x: limit lower=-3.141592653589793 upper=3.141592653589793 effort=10 velocity=10 -> lower=-3.141592653589793 upper=3.141592653589793 effort=10 velocity=1e+08
- joint passive_6_y: limit lower=-3.141592653589793 upper=3.141592653589793 effort=10 velocity=10 -> lower=-3.141592653589793 upper=3.141592653589793 effort=10 velocity=1e+08
- joint passive_6_z: limit lower=-3.141592653589793 upper=3.141592653589793 effort=10 velocity=10 -> lower=-3.141592653589793 upper=3.141592653589793 effort=10 velocity=1e+08
- joint passive_7_x: limit lower=-3.141592653589793 upper=3.141592653589793 effort=10 velocity=10 -> lower=-3.141592653589793 upper=3.141592653589793 effort=10 velocity=1e+08
- joint passive_7_y: limit lower=-3.141592653589793 upper=3.141592653589793 effort=10 velocity=10 -> lower=-3.141592653589793 upper=3.141592653589793 effort=10 velocity=1e+08
- joint passive_7_z: limit lower=-3.141592653589793 upper=3.141592653589793 effort=10 velocity=10 -> lower=-3.141592653589793 upper=3.141592653589793 effort=10 velocity=1e+08

Commit message: new mjcf and urdf

File: descriptions/reachy_mini/urdf/robot.urdf (robot description, URDF)
Before this commit: robot robot, 42 links, 41 joints
Links:
- removed link arm
- removed link arm_2
- removed link arm_3
- removed link arm_4
- removed link arm_5
- removed link ball
- removed link main_plate
- removed link plateform
- removed link rod
- removed link turning_bowl
- added link camera, mass 1e-9
- added link camera_optical, mass 1e-9
- added link dc15_a01_case_b_dummy, mass 0.391334; collision mesh filename=package://assets/dc15_a01_case_b_dummy.stl; collision mesh filename=package://assets/dc15_a01_case_b_dummy.stl
- added link pp00xxx_stewart_rod, mass 1e-09; collision mesh filename=package://assets/pp00xxx_stewart_rod.stl; collision mesh filename=package://assets/shape.stl
- added link pp01062_stewart_arm, mass 1e-09; collision mesh filename=package://assets/ball.stl; collision mesh filename=package://assets/pp01062_stewart_arm.stl
- added link pp01062_stewart_arm_2, mass 1e-09; collision mesh filename=package://assets/ball.stl; collision mesh filename=package://assets/pp01062_stewart_arm.stl
- added link pp01062_stewart_arm_3, mass 1e-09; collision mesh filename=package://assets/ball.stl; collision mesh filename=package://assets/pp01062_stewart_arm.stl
- added link pp01062_stewart_arm_4, mass 1e-09; collision mesh filename=package://assets/ball.stl; collision mesh filename=package://assets/pp01062_stewart_arm.stl
- added link pp01062_stewart_arm_5, mass 1e-09; collision mesh filename=package://assets/ball.stl; collision mesh filename=package://assets/pp01062_stewart_arm.stl
- added link pp01062_stewart_arm_6, mass 1e-09; collision mesh filename=package://assets/ball.stl; collision mesh filename=package://assets/pp01062_stewart_arm.stl
- added link pp01063_stewart_plateform, mass 0.109232; collision mesh filename=package://assets/ball.stl; collision mesh filename=package://assets/ball.stl
- added link pp01071_turning_bowl, mass 0.0947234; collision mesh filename=package://assets/pp01071_turning_bowl.stl; collision mesh filename=package://assets/pp01072_turning_end.stl
- link shape: geometry collision mesh filename=package://assets/pp00xxx_stewart_rod.stl; collision mesh filename=package://assets/shape.stl
- link shape_2: geometry collision mesh filename=package://assets/pp00xxx_stewart_rod.stl; collision mesh filename=package://assets/shape.stl
- link shape_3: geometry collision mesh filename=package://assets/pp00xxx_stewart_rod.stl; collision mesh filename=package://assets/shape.stl
- link shape_4: geometry collision mesh filename=package://assets/pp00xxx_stewart_rod.stl; collision mesh filename=package://assets/shape.stl
- link shape_5: geometry collision mesh filename=package://assets/pp00xxx_stewart_rod.stl; collision mesh filename=package://assets/shape.stl
- link test_antenna: mass 0.00463834 -> 0.00456766
- link test_antenna_body: mass 0.00463834 -> 0.00456766
Joints:
- added joint camera_frame: type fixed, parent pp01063_stewart_plateform, child camera, origin xyz=0.0244171 -0.0524 0.0147383 rpy=1.5708 0.523599 -8.01234e-18, axis 0 0 0
- added joint camera_optical_frame: type fixed, parent pp01063_stewart_plateform, child camera_optical, origin xyz=0.0244171 -0.0524 0.0147383 rpy=3.14159 1.0472 3.14159, axis 0 0 0
- joint 1: child arm -> pp01062_stewart_arm; origin xyz=0.0313706 0.0298975 -0.044785 rpy=-1.5708 -5.45775e-15 -1.0472 -> xyz=0.0317603 0.0301725 -0.03705 rpy=1.5708 7.95539e-16 2.0944; parent main_plate -> dc15_a01_case_b_dummy
- joint 2: child arm_2 -> pp01062_stewart_arm_2; origin xyz=0.0416206 0.012144 -0.044785 rpy=-1.5708 -5.45775e-15 -1.0472 -> xyz=0.0420103 0.012419 -0.03705 rpy=-1.5708 -1.05471e-15 -1.0472; parent main_plate -> dc15_a01_case_b_dummy
- joint 3: child arm_3 -> pp01062_stewart_arm_3; origin xyz=0.0102933 -0.0421165 -0.044785 rpy=1.5708 -3.34105e-15 1.49303e-15 -> xyz=0.01025 -0.0425915 -0.03705 rpy=1.5708 -2.77556e-16 3.14916e-16; parent main_plate -> dc15_a01_case_b_dummy
- joint 4: child ball -> pp01062_stewart_arm_4; origin xyz=-0.0102067 -0.0421165 -0.044785 rpy=-1.5708 -2.17603e-15 -3.14159 -> xyz=-0.01025 -0.0425915 -0.03705 rpy=-1.5708 4.44377e-15 3.14159; parent main_plate -> dc15_a01_case_b_dummy
- joint 5: child arm_4 -> pp01062_stewart_arm_5; origin xyz=-0.041534 0.012144 -0.044785 rpy=-1.5708 9.76173e-15 1.0472 -> xyz=-0.0420103 0.012419 -0.03705 rpy=1.5708 4.85252e-16 -2.0944; parent main_plate -> dc15_a01_case_b_dummy
- joint 6: child arm_5 -> pp01062_stewart_arm_6; origin xyz=-0.031284 0.0298975 -0.044785 rpy=-1.5708 9.76173e-15 1.0472 -> xyz=-0.0317603 0.0301725 -0.03705 rpy=-1.5708 1.05471e-15 1.0472; parent main_plate -> dc15_a01_case_b_dummy
- joint all_yaw: child main_plate -> dc15_a01_case_b_dummy; limit lower=-2.96706 upper=2.96706 effort=10 velocity=8 -> lower=-3.141592653589793 upper=3.141592653589793 effort=10 velocity=8; origin xyz=-0.00198261 3.46945e-18 0.0316 rpy=-3.14159 -3.15544e-30 1.5708 -> xyz=4.85723e-17 -5.60663e-19 0.0339 rpy=3.14159 -2.22045e-16 1.5708; parent turning_bowl -> pp01071_turning_bowl
- joint closing_1_1_frame: origin xyz=-0.0900003 -4.16334e-17 -1.04083e-16 rpy=-8.64204e-18 6.344e-15 -3.14159 -> xyz=-0.0900003 -2.77556e-17 -8.32667e-17 rpy=-3.14159 1.84488e-15 -3.14159; parent rod -> shape
- joint closing_1_2_frame: origin xyz=-0.0107081 -0.00281895 -0.0487017 rpy=2.47273 0.170541 -0.454 -> xyz=0.0249723 5.55112e-17 0.0432533 rpy=2.0944 -4.74456e-17 -1.5708; parent plateform -> pp01063_stewart_plateform
- joint closing_2_1_frame: origin xyz=-0.0900003 0 0 rpy=-6.98035e-17 -9.35855e-17 3.14159 -> xyz=0.0184723 5.55112e-17 0.0545117 rpy=-3.14159 1.0472 -3.66493e-30; parent shape -> pp01063_stewart_plateform
- joint closing_2_2_frame: origin xyz=-0.00746482 0.00694678 -0.056646 rpy=2.47273 0.170541 -0.454 -> xyz=-0.0900003 -2.77556e-17 2.08167e-17 rpy=3.14159 -5.94057e-16 -1.5708; parent plateform -> shape_2
- joint closing_3_1_frame: origin xyz=-0.0900003 -1.38778e-17 -2.70617e-16 rpy=-9.02091e-17 5.6271e-16 -3.14159 -> xyz=-0.0314723 2.77556e-17 0.0545117 rpy=-2.0944 -2.36516e-15 -1.5708; parent shape_2 -> pp01063_stewart_plateform
- joint closing_3_2_frame: origin xyz=0.0157039 0.0472846 -0.0384653 rpy=0.871822 -1.34723 0.257412 -> xyz=-0.0900003 0 1.31839e-16 rpy=-1.02731e-16 -1.66398e-15 3.14159; parent plateform -> shape_3
- joint closing_4_1_frame: origin xyz=-0.0900003 -1.38778e-17 -9.54098e-18 rpy=-7.37315e-16 2.73389e-16 3.14159 -> xyz=-0.0900003 2.08167e-16 3.46945e-18 rpy=-3.14159 2.0365e-19 3.14159; parent shape_3 -> shape_4
- joint closing_4_2_frame: origin xyz=0.0184911 0.0480184 -0.0257888 rpy=-0.871822 1.34723 -2.88418 -> xyz=-0.0379723 5.55112e-17 0.0432533 rpy=1.0472 -6.90096e-15 -1.5708; parent plateform -> pp01063_stewart_plateform
- joint closing_5_1_frame: origin xyz=-0.0900003 -1.38778e-17 -3.05311e-16 rpy=-5.60604e-16 3.49956e-15 3.14159 -> xyz=-0.0900003 1.38778e-16 6.93889e-18 rpy=-3.14159 -7.144e-17 -3.14159; parent shape_4 -> pp00xxx_stewart_rod
- joint closing_5_2_frame: origin xyz=0.00603053 0.0104995 0.00473221 rpy=2.95835 0.372577 -2.09215 -> xyz=-0.013 5.55112e-17 -5.55112e-17 rpy=-3.77194e-17 5.29636e-15 -1.5708; parent plateform -> pp01063_stewart_plateform
- joint head_frame: origin xyz=0.00367542 0.0183217 -0.0274783 rpy=-1.74312 -0.143141 -1.99997 -> xyz=-0.0134282 -0.0012 0.0365883 rpy=1.5708 0.523599 4.24373e-30; parent plateform -> pp01063_stewart_plateform
- joint left_antenna: origin xyz=0.0786202 0.0183429 -0.0976865 rpy=-0.242906 0.87314 -2.31329 -> xyz=-0.0161053 -0.0744 0.100068 rpy=-3.08341 -0.527253 0.0579647; parent plateform -> pp01063_stewart_plateform
- joint passive_1_x: origin xyz=-0.038 -1.80411e-16 -0.00768 rpy=-0.173384 -0.0202587 -2.05328 -> xyz=0.038 -2.77556e-17 -0.00768 rpy=0.0485766 -0.0258157 1.08824; parent arm -> pp01062_stewart_arm
- joint passive_1_y: origin xyz=6.93889e-18 -1.38778e-17 0 rpy=8.62746e-18 1.20021e-17 3.19976e-17 -> xyz=6.93889e-18 -1.38778e-17 0 rpy=6.20901e-17 1.31226e-17 -3.8231e-17
- joint passive_1_z: child rod -> shape; origin xyz=6.93889e-18 -1.38778e-17 0 rpy=8.62746e-18 1.20021e-17 3.19976e-17 -> xyz=6.93889e-18 -1.38778e-17 0 rpy=6.20901e-17 1.31226e-17 -3.8231e-17
- joint passive_2_x: origin xyz=0.038 6.52256e-16 -0.00768 rpy=-0.186454 -0.0202587 -1.08831 -> xyz=0.038 8.32667e-17 -0.00768 rpy=0.046409 -0.0258157 -1.08824; parent arm_2 -> pp01062_stewart_arm_2
- joint passive_2_y: origin xyz=6.93889e-18 0 0 rpy=-1.58342e-17 -1.2695e-17 -3.61667e-17 -> xyz=6.93889e-18 0 6.93889e-18 rpy=1.03529e-16 -2.76081e-18 1.06701e-17
- joint passive_2_z: child shape -> shape_2; origin xyz=6.93889e-18 0 0 rpy=-1.58342e-17 -1.2695e-17 -3.61667e-17 -> xyz=6.93889e-18 0 6.93889e-18 rpy=1.03529e-16 -2.76081e-18 1.06701e-17
- joint passive_3_x: origin xyz=0.038 0 -0.00768 rpy=2.99943 -0.0202587 1.08831 -> xyz=0.038 -4.16334e-17 -0.00768 rpy=3.06133 -0.0258157 1.08824; parent arm_3 -> pp01062_stewart_arm_3
- joint passive_3_y: origin xyz=6.93889e-18 0 3.46945e-18 rpy=-1.14555e-17 -7.10933e-18 1.4473e-17 -> xyz=1.38778e-17 0 0 rpy=-1.00225e-17 4.94486e-18 1.68244e-17
- joint passive_3_z: child shape_2 -> shape_3; origin xyz=6.93889e-18 0 3.46945e-18 rpy=-1.14555e-17 -7.10933e-18 1.4473e-17 -> xyz=1.38778e-17 0 0 rpy=-1.00225e-17 4.94486e-18 1.68244e-17
- joint passive_4_x: origin xyz=0.038 1.38778e-17 -0.00768 rpy=-2.75098 -0.0202587 -1.08831 -> xyz=0.038 2.77556e-17 -0.00768 rpy=-3.02327 -0.0258157 -1.08824; parent ball -> pp01062_stewart_arm_4
- joint passive_4_y: origin xyz=1.38778e-17 -1.38778e-17 -5.20417e-18 rpy=2.34572e-17 -1.42363e-18 -4.04804e-17 -> xyz=6.93889e-18 0 3.46945e-18 rpy=-5.32364e-18 3.35739e-18 2.46433e-17
- joint passive_4_z: child shape_3 -> shape_4; origin xyz=1.38778e-17 -1.38778e-17 -5.20417e-18 rpy=2.34572e-17 -1.42363e-18 -4.04804e-17 -> xyz=6.93889e-18 0 3.46945e-18 rpy=-5.32364e-18 3.35739e-18 2.46433e-17
- joint passive_5_x: origin xyz=-0.038 2.35922e-16 -0.00768 rpy=-2.7279 -0.0202587 -2.05328 -> xyz=0.038 -1.38778e-17 -0.00768 rpy=0.197132 -0.0258157 1.08824; parent arm_4 -> pp01062_stewart_arm_5
- joint passive_5_y: origin xyz=6.93889e-18 0 -1.38778e-17 rpy=2.80246e-17 -2.32495e-17 -3.77543e-17 -> xyz=0 0 0 rpy=-3.08493e-17 2.79333e-17 5.24089e-17
- joint passive_5_z: child shape_4 -> pp00xxx_stewart_rod; origin xyz=6.93889e-18 0 -1.38778e-17 rpy=2.80246e-17 -2.32495e-17 -3.77543e-17 -> xyz=0 0 0 rpy=-3.08493e-17 2.79333e-17 5.24089e-17
- joint passive_6_x: origin xyz=0.038 -2.498e-16 -0.00768 rpy=-2.72876 -0.0202587 -1.08831 -> xyz=0.038 2.77556e-17 -0.00768 rpy=0.0463478 -0.0258157 -1.08824; parent arm_5 -> pp01062_stewart_arm_6
- joint passive_6_y: origin xyz=-2.08167e-17 1.38778e-17 1.6263e-18 rpy=-2.45872e-17 1.38232e-19 7.28361e-17 -> xyz=6.93889e-18 0 0 rpy=9.77399e-17 3.28422e-18 1.01949e-16
- joint passive_6_z: origin xyz=-2.08167e-17 1.38778e-17 1.6263e-18 rpy=-2.45872e-17 1.38232e-19 7.28361e-17 -> xyz=6.93889e-18 0 0 rpy=9.77399e-17 3.28422e-18 1.01949e-16
- joint passive_7_x: origin xyz=-0.0900003 -2.77556e-17 7.80626e-18 rpy=3.14159 -2.94505e-16 -3.14159 -> xyz=-0.0900003 1.88738e-15 -2.08167e-17 rpy=-3.14025 0.0530311 1.08768
- joint passive_7_y: origin xyz=0 1.38778e-17 -7.48099e-18 rpy=-1.94479e-17 1.88775e-18 6.89749e-18 -> xyz=-8.67362e-19 2.77556e-17 0 rpy=-1.00928e-30 6.45118e-17 -2.11395e-31
- joint passive_7_z: child plateform -> pp01063_stewart_plateform; origin xyz=0 1.38778e-17 -7.48099e-18 rpy=-1.94479e-17 1.88775e-18 6.89749e-18 -> xyz=-8.67362e-19 2.77556e-17 0 rpy=-1.00928e-30 6.45118e-17 -2.11395e-31
- joint right_antenna: origin xyz=0.101086 0.024257 0.00448913 rpy=-3.0252 1.213 1.08209 -> xyz=-0.0697422 -0.0744 0.00716666 rpy=-1.5708 -1.40009 -1.48353; parent plateform -> pp01063_stewart_plateform

Commit message: decimating meshes a little more to run faster in mujoco

File: descriptions/reachy_mini/urdf/robot.urdf (robot description, URDF)
Before this commit: robot robot, 44 links, 43 joints
Links:
- link dc15_a01_case_b_dummy: mass 0.391334 -> 0.443795
- link pp00xxx_stewart_rod: mass 1e-09 -> 0.00355525
- link pp01062_stewart_arm: mass 1e-09 -> 0.00272417
- link pp01062_stewart_arm_2: mass 1e-09 -> 0.00272417
- link pp01062_stewart_arm_3: mass 1e-09 -> 0.00272417
- link pp01062_stewart_arm_4: mass 1e-09 -> 0.00272417
- link pp01062_stewart_arm_5: mass 1e-09 -> 0.00272417
- link pp01062_stewart_arm_6: mass 1e-09 -> 0.00272417
- link pp01063_stewart_plateform: mass 0.109232 -> 0.168092
- link shape: mass 1e-09 -> 0.00355525
- link shape_2: mass 1e-09 -> 0.00355525
- link shape_3: mass 1e-09 -> 0.00355525
- link shape_4: mass 1e-09 -> 0.00355525
- link shape_5: mass 1e-09 -> 0.00355525

Commit message: inverting stewart and antennas dofs in onshape, should now match real robot

File: descriptions/reachy_mini/urdf/robot.urdf (robot description, URDF)
Before this commit: robot robot, 44 links, 43 joints
Joints:
- joint 1: origin xyz=0.0317603 0.0301725 -0.03705 rpy=1.5708 7.95539e-16 2.0944 -> xyz=0.0317603 0.0301725 -0.03705 rpy=-1.5708 7.95539e-16 2.0944
- joint 2: origin xyz=0.0420103 0.012419 -0.03705 rpy=-1.5708 -1.05471e-15 -1.0472 -> xyz=0.0420103 0.012419 -0.03705 rpy=1.5708 -1.05471e-15 -1.0472
- joint 3: origin xyz=0.01025 -0.0425915 -0.03705 rpy=1.5708 -2.77556e-16 3.14916e-16 -> xyz=0.01025 -0.0425915 -0.03705 rpy=-1.5708 -2.77556e-16 3.14916e-16
- joint 4: origin xyz=-0.01025 -0.0425915 -0.03705 rpy=-1.5708 4.44377e-15 3.14159 -> xyz=-0.01025 -0.0425915 -0.03705 rpy=1.5708 4.44377e-15 3.14159
- joint 5: origin xyz=-0.0420103 0.012419 -0.03705 rpy=1.5708 4.85252e-16 -2.0944 -> xyz=-0.0420103 0.012419 -0.03705 rpy=-1.5708 4.85252e-16 -2.0944
- joint 6: origin xyz=-0.0317603 0.0301725 -0.03705 rpy=-1.5708 1.05471e-15 1.0472 -> xyz=-0.0317603 0.0301725 -0.03705 rpy=1.5708 1.05471e-15 1.0472
- joint left_antenna: origin xyz=-0.0161053 -0.0744 0.100068 rpy=-3.08341 -0.527253 0.0579647 -> xyz=-0.0161053 -0.0744 0.100068 rpy=0.0581863 -0.527253 0.0579647
- joint passive_1_x: origin xyz=0.038 -2.77556e-17 -0.00768 rpy=0.0485766 -0.0258157 1.08824 -> xyz=0.038 2.77556e-17 0.00768 rpy=-3.09302 0.0258157 -1.08824
- joint passive_2_x: origin xyz=0.038 8.32667e-17 -0.00768 rpy=0.046409 -0.0258157 -1.08824 -> xyz=0.038 -8.32667e-17 0.00768 rpy=-3.09518 0.0258157 1.08824
- joint passive_3_x: origin xyz=0.038 -4.16334e-17 -0.00768 rpy=3.06133 -0.0258157 1.08824 -> xyz=0.038 4.16334e-17 0.00768 rpy=-0.0802622 0.0258157 -1.08824
- joint passive_4_x: origin xyz=0.038 2.77556e-17 -0.00768 rpy=-3.02327 -0.0258157 -1.08824 -> xyz=0.038 -2.77556e-17 0.00768 rpy=0.118327 0.0258157 1.08824
- joint passive_5_x: origin xyz=0.038 -1.38778e-17 -0.00768 rpy=0.197132 -0.0258157 1.08824 -> xyz=0.038 1.38778e-17 0.00768 rpy=-2.94446 0.0258157 -1.08824
- joint passive_6_x: origin xyz=0.038 2.77556e-17 -0.00768 rpy=0.0463478 -0.0258157 -1.08824 -> xyz=0.038 -2.77556e-17 0.00768 rpy=-3.09524 0.0258157 1.08824
- joint right_antenna: origin xyz=-0.0697422 -0.0744 0.00716666 rpy=-1.5708 -1.40009 -1.48353 -> xyz=-0.0697422 -0.0744 0.00716666 rpy=1.5708 -1.40009 -1.48353
