Commit message: a biot more testing of the QP problems and added some additional constraints

File: src/reachy_mini/descriptions/reachy_mini/urdf/robot.urdf (robot description, URDF)
Before this commit: robot robot, 44 links, 43 joints
Links:
- added link dummy_torso_yaw; visual box size=0 0 0
Joints:
- added joint dummy_yaw: type fixed, parent dc15_a01_case_b_dummy, child dummy_torso_yaw, origin xyz=0 0 0 rpy=3.14 0 1.57, axis 0 0 1

Commit message: better velocity limit from teh xl330 datasheet

File: src/reachy_mini/descriptions/reachy_mini/urdf/robot.urdf (robot description, URDF)
Before this commit: robot robot, 45 links, 44 joints
Joints:
- joint 1: limit lower=-1.39626 upper=1.39626 effort=10 velocity=8 -> lower=-1.39626 upper=1.39626 effort=10 velocity=10
- joint 2: limit lower=-1.39626 upper=1.39626 effort=10 velocity=8 -> lower=-1.39626 upper=1.39626 effort=10 velocity=10
- joint 3: limit lower=-1.39626 upper=1.39626 effort=10 velocity=8 -> lower=-1.39626 upper=1.39626 effort=10 velocity=10
- joint 4: limit lower=-1.39626 upper=1.39626 effort=10 velocity=8 -> lower=-1.39626 upper=1.39626 effort=10 velocity=10
- joint 5: limit lower=-1.39626 upper=1.39626 effort=10 velocity=8 -> lower=-1.39626 upper=1.39626 effort=10 velocity=10
- joint 6: limit lower=-1.39626 upper=1.39626 effort=10 velocity=8 -> lower=-1.39626 upper=1.39626 effort=10 velocity=10
- joint all_yaw: limit lower=-3.141592653589793 upper=3.141592653589793 effort=10 velocity=8 -> lower=-3.141592653589793 upper=3.141592653589793 effort=10 velocity=10
- joint left_antenna: limit lower=-3.141592653589793 upper=3.141592653589793 effort=10 velocity=8 -> lower=-3.141592653589793 upper=3.141592653589793 effort=10 velocity=10
- joint right_antenna: limit lower=-3.141592653589793 upper=3.141592653589793 effort=10 velocity=8 -> lower=-3.141592653589793 upper=3.141592653589793 effort=10 velocity=10

Commit message: increase the velocities atrificially

File: src/reachy_mini/descriptions/reachy_mini/urdf/robot.urdf (robot description, URDF)
Before this commit: robot robot, 45 links, 44 joints
Joints:
- joint 1: limit lower=-1.39626 upper=1.39626 effort=10 velocity=10 -> lower=-1.39626 upper=1.39626 effort=10 velocity=20
- joint 2: limit lower=-1.39626 upper=1.39626 effort=10 velocity=10 -> lower=-1.39626 upper=1.39626 effort=10 velocity=20
- joint 3: limit lower=-1.39626 upper=1.39626 effort=10 velocity=10 -> lower=-1.39626 upper=1.39626 effort=10 velocity=20
- joint 4: limit lower=-1.39626 upper=1.39626 effort=10 velocity=10 -> lower=-1.39626 upper=1.39626 effort=10 velocity=20
- joint 5: limit lower=-1.39626 upper=1.39626 effort=10 velocity=10 -> lower=-1.39626 upper=1.39626 effort=10 velocity=20
- joint 6: limit lower=-1.39626 upper=1.39626 effort=10 velocity=10 -> lower=-1.39626 upper=1.39626 effort=10 velocity=20
- joint all_yaw: limit lower=-3.141592653589793 upper=3.141592653589793 effort=10 velocity=10 -> lower=-3.141592653589793 upper=3.141592653589793 effort=10 velocity=20
- joint left_antenna: limit lower=-3.141592653589793 upper=3.141592653589793 effort=10 velocity=10 -> lower=-3.141592653589793 upper=3.141592653589793 effort=10 velocity=20
- joint right_antenna: limit lower=-3.141592653589793 upper=3.141592653589793 effort=10 velocity=10 -> lower=-3.141592653589793 upper=3.141592653589793 effort=10 velocity=20

Commit message: max speed in software

File: src/reachy_mini/descriptions/reachy_mini/urdf/robot.urdf (robot description, URDF)
Before this commit: robot robot, 45 links, 44 joints
Joints:
- joint 1: limit lower=-1.39626 upper=1.39626 effort=10 velocity=20 -> lower=-1.39626 upper=1.39626 effort=10 velocity=10
- joint 2: limit lower=-1.39626 upper=1.39626 effort=10 velocity=20 -> lower=-1.39626 upper=1.39626 effort=10 velocity=10
- joint 3: limit lower=-1.39626 upper=1.39626 effort=10 velocity=20 -> lower=-1.39626 upper=1.39626 effort=10 velocity=10
- joint 4: limit lower=-1.39626 upper=1.39626 effort=10 velocity=20 -> lower=-1.39626 upper=1.39626 effort=10 velocity=10
- joint 5: limit lower=-1.39626 upper=1.39626 effort=10 velocity=20 -> lower=-1.39626 upper=1.39626 effort=10 velocity=10
- joint 6: limit lower=-1.39626 upper=1.39626 effort=10 velocity=20 -> lower=-1.39626 upper=1.39626 effort=10 velocity=10
- joint all_yaw: limit lower=-3.141592653589793 upper=3.141592653589793 effort=10 velocity=20 -> lower=-3.141592653589793 upper=3.141592653589793 effort=10 velocity=10
- joint left_antenna: limit lower=-3.141592653589793 upper=3.141592653589793 effort=10 velocity=20 -> lower=-3.141592653589793 upper=3.141592653589793 effort=10 velocity=10
- joint right_antenna: limit lower=-3.141592653589793 upper=3.141592653589793 effort=10 velocity=20 -> lower=-3.141592653589793 upper=3.141592653589793 effort=10 velocity=10

Commit message: update URDF and MJCF. Placo Kinematics seems to work (need more testing). Rust and NN kinematics not working yet.

File: src/reachy_mini/descriptions/reachy_mini/urdf/robot.urdf (robot description, URDF)
Before this commit: robot robot, 45 links, 44 joints
Links:
- removed link dc15_a01_case_b_dummy
- removed link pp00xxx_stewart_rod
- removed link pp01062_stewart_arm
- removed link pp01062_stewart_arm_2
- removed link pp01062_stewart_arm_3
- removed link pp01062_stewart_arm_4
- removed link pp01062_stewart_arm_5
- removed link pp01062_stewart_arm_6
- removed link pp01063_stewart_plateform
- removed link pp01071_turning_bowl
- removed link shape
- removed link shape_2
- removed link shape_3
- removed link shape_4
- removed link shape_5
- removed link test_antenna
- removed link test_antenna_body
- added link body_down_3dprint, mass 0.78209; collision mesh filename=package://assets/5w_speaker.stl; collision mesh filename=package://assets/b3b_eh.stl
- added link body_foot_3dprint, mass 0.0617881; collision mesh filename=package://assets/body_foot_3dprint.stl; collision mesh filename=package://assets/body_turning_3dprint.stl
- added link dc15_a01_horn_dummy, mass 0.00366675; collision mesh filename=package://assets/dc15_a01_horn_dummy.stl; collision mesh filename=package://assets/mp01062_stewart_arm_3.stl
- added link dc15_a01_horn_dummy_2, mass 0.00366675; collision mesh filename=package://assets/dc15_a01_horn_dummy.stl; collision mesh filename=package://assets/mp01062_stewart_arm_3.stl
- added link dc15_a01_horn_dummy_3, mass 0.00366675; collision mesh filename=package://assets/dc15_a01_horn_dummy.stl; collision mesh filename=package://assets/mp01062_stewart_arm_3.stl
- added link dc15_a01_horn_dummy_4, mass 0.00366675; collision mesh filename=package://assets/dc15_a01_horn_dummy.stl; collision mesh filename=package://assets/mp01062_stewart_arm_3.stl
- added link dc15_a01_horn_dummy_5, mass 0.00366675; collision mesh filename=package://assets/dc15_a01_horn_dummy.stl; collision mesh filename=package://assets/mp01062_stewart_arm_3.stl
- added link dc15_a01_horn_dummy_6, mass 0.00366675; collision mesh filename=package://assets/dc15_a01_horn_dummy.stl; collision mesh filename=package://assets/mp01062_stewart_arm_3.stl
- added link dc15_a01_horn_dummy_7, mass 0.0105926; collision mesh filename=package://assets/antenna.stl; collision mesh filename=package://assets/antenna_body_3dprint.stl
- added link dc15_a01_horn_dummy_8, mass 0.0105926; collision mesh filename=package://assets/antenna.stl; collision mesh filename=package://assets/antenna_body_3dprint.stl
- added link stewart_link_rod, mass 0.00503424; collision mesh filename=package://assets/stewart_link_rod.stl; visual mesh filename=package://assets/stewart_link_rod.stl
- added link stewart_link_rod_2, mass 0.00503424; collision mesh filename=package://assets/stewart_link_rod.stl; visual mesh filename=package://assets/stewart_link_rod.stl
- added link stewart_link_rod_3, mass 0.00503424; collision mesh filename=package://assets/stewart_link_rod.stl; visual mesh filename=package://assets/stewart_link_rod.stl
- added link stewart_link_rod_4, mass 0.00503424; collision mesh filename=package://assets/stewart_link_rod.stl; visual mesh filename=package://assets/stewart_link_rod.stl
- added link stewart_link_rod_5, mass 0.00503424; collision mesh filename=package://assets/stewart_link_rod.stl; visual mesh filename=package://assets/stewart_link_rod.stl
- added link stewart_link_rod_6, mass 0.00503424; collision mesh filename=package://assets/stewart_link_rod.stl; visual mesh filename=package://assets/stewart_link_rod.stl
- added link xl_330, mass 0.259259; collision mesh filename=package://assets/antenna_holder_l_3dprint.stl; collision mesh filename=package://assets/antenna_holder_r_3dprint.stl
Joints:
- removed joint 1
- removed joint 2
- removed joint 3
- removed joint 4
- removed joint 5
- removed joint 6
- removed joint all_yaw
- added joint stewart_1: type revolute, parent body_down_3dprint, child dc15_a01_horn_dummy, origin xyz=-0.0328112 -0.0304906 -0.0418333 rpy=-1.5708 3.05628e-14 -1.0472, axis 0 0 1, limit lower=-3.141592653589793 upper=3.141592653589793 effort=10 velocity=8
- added joint stewart_2: type revolute, parent body_down_3dprint, child dc15_a01_horn_dummy_2, origin xyz=-0.0428112 -0.01317 -0.0418333 rpy=-1.5708 6.75017e-15 -1.0472, axis 0 0 1, limit lower=-3.141592653589793 upper=3.141592653589793 effort=10 velocity=8
- added joint stewart_3: type revolute, parent body_down_3dprint, child dc15_a01_horn_dummy_3, origin xyz=-0.01 0.0436606 -0.0418333 rpy=1.5708 1.5708 0, axis 0 0 1, limit lower=-3.141592653589793 upper=3.141592653589793 effort=10 velocity=8
- added joint stewart_4: type revolute, parent body_down_3dprint, child dc15_a01_horn_dummy_4, origin xyz=0.01 0.0436606 -0.0418333 rpy=1.5708 1.5708 0, axis 0 0 1, limit lower=-3.141592653589793 upper=3.141592653589793 effort=10 velocity=8
- added joint stewart_5: type revolute, parent body_down_3dprint, child dc15_a01_horn_dummy_5, origin xyz=0.0428112 -0.01317 -0.0418333 rpy=-2.61799 1.5708 0, axis 0 0 1, limit lower=-3.141592653589793 upper=3.141592653589793 effort=10 velocity=8
- added joint stewart_6: type revolute, parent body_down_3dprint, child dc15_a01_horn_dummy_6, origin xyz=0.0328112 -0.0304906 -0.0418333 rpy=-1.5708 1.11952e-14 1.0472, axis 0 0 1, limit lower=-3.141592653589793 upper=3.141592653589793 effort=10 velocity=8
- added joint yaw_body: type revolute, parent body_foot_3dprint, child body_down_3dprint, origin xyz=-2.45997e-07 6.93889e-18 0.0348 rpy=-3.14159 6.78125e-28 -1.5708, axis 0 0 1, limit lower=-3.141592653589793 upper=3.141592653589793 effort=10 velocity=8
- joint camera_frame: origin xyz=0.0244171 -0.0524 0.0147383 rpy=1.5708 0.523599 -8.01234e-18 -> xyz=-0.0367778 -0.0471665 0.00283045 rpy=1.69996 0.547922 -1.07174; parent pp01063_stewart_plateform -> xl_330
- joint camera_optical_frame: origin xyz=0.0244171 -0.0524 0.0147383 rpy=3.14159 1.0472 3.14159 -> xyz=-0.0367778 -0.0471665 0.00283045 rpy=2.93358 1.00937 1.82549; parent pp01063_stewart_plateform -> xl_330
- joint closing_1_1_frame: origin xyz=-0.0900003 -2.77556e-17 -8.32667e-17 rpy=-3.14159 1.84488e-15 -3.14159 -> xyz=0.085 -1.38778e-17 -6.93889e-18 rpy=-1.89585e-17 -5.12506e-17 5.13924e-17; parent shape -> stewart_link_rod
- joint closing_1_2_frame: origin xyz=0.0249723 5.55112e-17 0.0432533 rpy=2.0944 -4.74456e-17 -1.5708 -> xyz=0.00583863 -0.022426 0.0368459 rpy=-2.91303 1.06415 -0.938629; parent pp01063_stewart_plateform -> xl_330
- joint closing_2_1_frame: origin xyz=0.0184723 5.55112e-17 0.0545117 rpy=-3.14159 1.0472 -3.66493e-30 -> xyz=-0.014684 -0.0833865 -0.00748861 rpy=3.07468 -0.0882156 1.39649; parent pp01063_stewart_plateform -> stewart_link_rod_2
- joint closing_2_2_frame: origin xyz=-0.0900003 -2.77556e-17 2.08167e-17 rpy=3.14159 -5.94057e-16 -1.5708 -> xyz=0.00182437 -0.0169454 0.0490871 rpy=-2.91303 1.06415 -0.938629; parent shape_2 -> xl_330
- joint closing_3_1_frame: origin xyz=-0.0314723 2.77556e-17 0.0545117 rpy=-2.0944 -2.36516e-15 -1.5708 -> xyz=-0.085 -6.93889e-18 0 rpy=-2.43112e-17 2.25632e-17 2.00133e-17; parent pp01063_stewart_plateform -> stewart_link_rod_3
- joint closing_3_2_frame: origin xyz=-0.0900003 0 1.31839e-16 rpy=-1.02731e-16 -1.66398e-15 3.14159 -> xyz=-0.016495 0.0225206 0.0503005 rpy=-2.93358 -1.00937 -1.3161; parent shape_3 -> xl_330
- joint closing_4_1_frame: origin xyz=-0.0900003 2.08167e-16 3.46945e-18 rpy=-3.14159 2.0365e-19 3.14159 -> xyz=-0.085 0 0 rpy=3.17368e-18 -3.23103e-18 -2.7013e-17; parent shape_4 -> stewart_link_rod_4
- joint closing_4_2_frame: origin xyz=-0.0379723 5.55112e-17 0.0432533 rpy=1.0472 -6.90096e-15 -1.5708 -> xyz=-0.0183729 0.0297336 0.0384495 rpy=-2.93358 -1.00937 -1.3161; parent pp01063_stewart_plateform -> xl_330
- joint closing_5_1_frame: origin xyz=-0.0900003 1.38778e-16 6.93889e-18 rpy=-3.14159 -7.144e-17 -3.14159 -> xyz=-0.085 0 0 rpy=-3.0015e-19 1.3471e-17 1.28245e-17; parent pp00xxx_stewart_rod -> stewart_link_rod_5
- joint closing_5_2_frame: origin xyz=-0.013 5.55112e-17 -5.55112e-17 rpy=-3.77194e-17 5.29636e-15 -1.5708 -> xyz=-0.00589217 0.0126937 0.00039027 rpy=-3.11354 -0.110171 0.431499; parent pp01063_stewart_plateform -> xl_330
- joint dummy_yaw: parent dc15_a01_case_b_dummy -> body_down_3dprint
- joint head_frame: origin xyz=-0.0134282 -0.0012 0.0365883 rpy=1.5708 0.523599 4.24373e-30 -> xyz=-0.00551617 0.00426275 0.0291789 rpy=1.69996 0.547922 -1.07174; parent pp01063_stewart_plateform -> xl_330
- joint left_antenna: child test_antenna_body -> dc15_a01_horn_dummy_8; limit lower=-3.141592653589793 upper=3.141592653589793 effort=10 velocity=10 -> lower=-3.141592653589793 upper=3.141592653589793 effort=10 velocity=8; origin xyz=-0.0161053 -0.0744 0.100068 rpy=0.0581863 -0.527253 0.0579647 -> xyz=-0.078553 -0.0250168 0.0845885 rpy=2.94387 0.505067 2.01001; parent pp01063_stewart_plateform -> xl_330
- joint passive_1_x: origin xyz=0.038 2.77556e-17 0.00768 rpy=-3.09302 0.0258157 -1.08824 -> xyz=0.0327739 0.0229319 0.007 rpy=-0.129033 -0.0882156 2.00701; parent pp01062_stewart_arm -> dc15_a01_horn_dummy
- joint passive_1_y: origin xyz=6.93889e-18 -1.38778e-17 0 rpy=6.20901e-17 1.31226e-17 -3.8231e-17 -> xyz=0 0 -6.93889e-18 rpy=-1.89585e-17 -5.12506e-17 5.13924e-17
- joint passive_1_z: child shape -> stewart_link_rod; origin xyz=6.93889e-18 -1.38778e-17 0 rpy=6.20901e-17 1.31226e-17 -3.8231e-17 -> xyz=0 0 -6.93889e-18 rpy=-1.89585e-17 -5.12506e-17 5.13924e-17
- joint passive_2_x: origin xyz=0.038 -8.32667e-17 0.00768 rpy=-3.09518 0.0258157 1.08824 -> xyz=-0.0327739 0.0229319 0.007 rpy=-3.14159 2.27308e-16 -0.610524; parent pp01062_stewart_arm_2 -> dc15_a01_horn_dummy_2
- joint passive_2_y: origin xyz=6.93889e-18 0 6.93889e-18 rpy=1.03529e-16 -2.76081e-18 1.06701e-17 -> xyz=0 6.93889e-18 6.93889e-18 rpy=3.32777e-18 -2.35601e-17 -9.45252e-18
- joint passive_2_z: child shape_2 -> stewart_link_rod_2; origin xyz=6.93889e-18 0 6.93889e-18 rpy=1.03529e-16 -2.76081e-18 1.06701e-17 -> xyz=0 6.93889e-18 6.93889e-18 rpy=3.32777e-18 -2.35601e-17 -9.45252e-18
- joint passive_3_x: origin xyz=0.038 4.16334e-17 0.00768 rpy=-0.0802622 0.0258157 -1.08824 -> xyz=0.0229319 -0.0327739 0.007 rpy=0.365063 0.0882156 -2.70538; parent pp01062_stewart_arm_3 -> dc15_a01_horn_dummy_3
- joint passive_3_y: origin xyz=1.38778e-17 0 0 rpy=-1.00225e-17 4.94486e-18 1.68244e-17 -> xyz=0 0 0 rpy=-2.43112e-17 2.25632e-17 2.00133e-17
- joint passive_3_z: child shape_3 -> stewart_link_rod_3; origin xyz=1.38778e-17 0 0 rpy=-1.00225e-17 4.94486e-18 1.68244e-17 -> xyz=0 0 0 rpy=-2.43112e-17 2.25632e-17 2.00133e-17
- joint passive_4_x: origin xyz=0.038 -2.77556e-17 0.00768 rpy=0.118327 0.0258157 1.08824 -> xyz=0.0229319 0.0327739 0.007 rpy=-0.077578 0.0882156 2.70538; parent pp01062_stewart_arm_4 -> dc15_a01_horn_dummy_4
- joint passive_4_y: origin xyz=6.93889e-18 0 3.46945e-18 rpy=-5.32364e-18 3.35739e-18 2.46433e-17 -> xyz=1.38778e-17 0 0 rpy=3.17368e-18 -3.23103e-18 -2.7013e-17
- joint passive_4_z: child shape_4 -> stewart_link_rod_4; origin xyz=6.93889e-18 0 3.46945e-18 rpy=-5.32364e-18 3.35739e-18 2.46433e-17 -> xyz=1.38778e-17 0 0 rpy=3.17368e-18 -3.23103e-18 -2.7013e-17
- joint passive_5_x: origin xyz=0.038 1.38778e-17 0.00768 rpy=-2.94446 0.0258157 -1.08824 -> xyz=0.0229319 -0.0327739 0.007 rpy=0.11547 0.0882156 -2.70538; parent pp01062_stewart_arm_5 -> dc15_a01_horn_dummy_5
- joint passive_5_y: origin xyz=0 0 0 rpy=-3.08493e-17 2.79333e-17 5.24089e-17 -> xyz=0 0 0 rpy=-3.0015e-19 1.3471e-17 1.28245e-17
- joint passive_5_z: child pp00xxx_stewart_rod -> stewart_link_rod_5; origin xyz=0 0 0 rpy=-3.08493e-17 2.79333e-17 5.24089e-17 -> xyz=0 0 0 rpy=-3.0015e-19 1.3471e-17 1.28245e-17
- joint passive_6_x: origin xyz=0.038 -2.77556e-17 0.00768 rpy=-3.09524 0.0258157 1.08824 -> xyz=-0.0327739 0.0229319 0.007 rpy=3.06981 0.0882156 -2.00701; parent pp01062_stewart_arm_6 -> dc15_a01_horn_dummy_6
- joint passive_6_y: origin xyz=6.93889e-18 0 0 rpy=9.77399e-17 3.28422e-18 1.01949e-16 -> xyz=-2.77556e-17 -1.38778e-17 0 rpy=-2.80507e-17 2.33044e-18 5.49106e-18
- joint passive_6_z: child shape_5 -> stewart_link_rod_6; origin xyz=6.93889e-18 0 0 rpy=9.77399e-17 3.28422e-18 1.01949e-16 -> xyz=-2.77556e-17 -1.38778e-17 0 rpy=-2.80507e-17 2.33044e-18 5.49106e-18
- joint passive_7_x: origin xyz=-0.0900003 1.88738e-15 -2.08167e-17 rpy=-3.14025 0.0530311 1.08768 -> xyz=-0.085 -1.38778e-17 6.93889e-18 rpy=3.14159 2.33044e-18 5.49106e-18; parent shape_5 -> stewart_link_rod_6
- joint passive_7_y: origin xyz=-8.67362e-19 2.77556e-17 0 rpy=-1.00928e-30 6.45118e-17 -2.11395e-31 -> xyz=-2.77556e-17 0 -6.93889e-18 rpy=-2.80507e-17 -2.33044e-18 -5.49106e-18
- joint passive_7_z: child pp01063_stewart_plateform -> xl_330; origin xyz=-8.67362e-19 2.77556e-17 0 rpy=-1.00928e-30 6.45118e-17 -2.11395e-31 -> xyz=-2.77556e-17 0 -6.93889e-18 rpy=-2.80507e-17 -2.33044e-18 -5.49106e-18
- joint right_antenna: child test_antenna -> dc15_a01_horn_dummy_7; limit lower=-3.141592653589793 upper=3.141592653589793 effort=10 velocity=10 -> lower=-3.141592653589793 upper=3.141592653589793 effort=10 velocity=8; origin xyz=-0.0697422 -0.0744 0.00716666 rpy=1.5708 -1.40009 -1.48353 -> xyz=-0.0925548 0.0287641 -0.00377325 rpy=1.66493 1.39725 0.631412; parent pp01063_stewart_plateform -> xl_330
