Commit message: rust kin works, but had to set the arms zeros at 90°. Not final

File: src/reachy_mini/descriptions/reachy_mini/urdf/robot.urdf (robot description, URDF)
Before this commit: robot robot, 45 links, 44 joints
Joints:
- joint camera_frame: origin xyz=-0.0367778 -0.0471665 0.00283045 rpy=1.69996 0.547922 -1.07174 -> xyz=-0.0321159 -0.05047 0.00257878 rpy=1.70724 0.544115 -0.97213
- joint camera_optical_frame: origin xyz=-0.0367778 -0.0471665 0.00283045 rpy=2.93358 1.00937 1.82549 -> xyz=-0.0321159 -0.05047 0.00257878 rpy=2.92045 1.01151 1.9102
- joint closing_1_1_frame: origin xyz=0.085 -1.38778e-17 -6.93889e-18 rpy=-1.89585e-17 -5.12506e-17 5.13924e-17 -> xyz=0.085 -1.38778e-17 -6.93889e-18 rpy=-1.1607e-16 3.42669e-17 4.62147e-17
- joint closing_1_2_frame: origin xyz=0.00583863 -0.022426 0.0368459 rpy=-2.91303 1.06415 -0.938629 -> xyz=0.00768882 -0.0217774 0.0368953 rpy=-2.90143 1.05953 -0.832675
- joint closing_2_1_frame: origin xyz=-0.014684 -0.0833865 -0.00748861 rpy=3.07468 -0.0882156 1.39649 -> xyz=0.043 -0.0729378 -0.00748861 rpy=3.06617 -0.0882156 2.10349
- joint closing_2_2_frame: origin xyz=0.00182437 -0.0169454 0.0490871 rpy=-2.91303 1.06415 -0.938629 -> xyz=0.00307947 -0.0167102 0.049105 rpy=-2.90143 1.05953 -0.832675
- joint closing_3_1_frame: origin xyz=-0.085 -6.93889e-18 0 rpy=-2.43112e-17 2.25632e-17 2.00133e-17 -> xyz=-0.085 0 -1.38778e-17 rpy=4.65239e-19 -4.2966e-17 1.0182e-17
- joint closing_3_2_frame: origin xyz=-0.016495 0.0225206 0.0503005 rpy=-2.93358 -1.00937 -1.3161 -> xyz=-0.0189403 0.0208215 0.050171 rpy=-2.92045 -1.01151 -1.23139
- joint closing_4_1_frame: origin xyz=-0.085 0 0 rpy=3.17368e-18 -3.23103e-18 -2.7013e-17 -> xyz=-0.085 -1.38778e-17 0 rpy=2.88217e-18 2.28461e-18 -8.3094e-17
- joint closing_4_2_frame: origin xyz=-0.0183729 0.0297336 0.0384495 rpy=-2.93358 -1.00937 -1.3161 -> xyz=-0.0214133 0.0278259 0.0383042 rpy=-2.92045 -1.01151 -1.23139
- joint closing_5_1_frame: origin xyz=-0.085 0 0 rpy=-3.0015e-19 1.3471e-17 1.28245e-17 -> xyz=-0.085 -2.77556e-17 1.38778e-17 rpy=-1.54617e-17 2.86037e-17 -1.44876e-17
- joint closing_5_2_frame: origin xyz=-0.00589217 0.0126937 0.00039027 rpy=-3.11354 -0.110171 0.431499 -> xyz=-0.00708235 0.0120716 0.000342873 rpy=-3.11693 -0.116645 0.52771
- joint head_frame: origin xyz=-0.00551617 0.00426275 0.0291789 rpy=1.69996 0.547922 -1.07174 -> xyz=-0.00611127 0.00370522 0.0291364 rpy=1.70724 0.544115 -0.97213
- joint left_antenna: origin xyz=-0.078553 -0.0250168 0.0845885 rpy=2.94387 0.505067 2.01001 -> xyz=-0.0764135 -0.0324475 0.0840224 rpy=2.93649 0.508471 2.10225
- joint passive_1_x: origin xyz=0.0327739 0.0229319 0.007 rpy=-0.129033 -0.0882156 2.00701 -> xyz=0.04 -1.6545e-10 0.007 rpy=-0.13754 -0.0882156 2.10349
- joint passive_1_y: origin xyz=0 0 -6.93889e-18 rpy=-1.89585e-17 -5.12506e-17 5.13924e-17 -> xyz=-1.38778e-17 0 -6.93889e-18 rpy=-1.1607e-16 3.42669e-17 4.62147e-17
- joint passive_1_z: origin xyz=0 0 -6.93889e-18 rpy=-1.89585e-17 -5.12506e-17 5.13924e-17 -> xyz=-1.38778e-17 0 -6.93889e-18 rpy=-1.1607e-16 3.42669e-17 4.62147e-17
- joint passive_2_x: origin xyz=-0.0327739 0.0229319 0.007 rpy=-3.14159 2.27308e-16 -0.610524 -> xyz=0.04 8.32667e-17 0.007 rpy=-3.14159 -9.64904e-17 -3.14159
- joint passive_2_y: origin xyz=0 6.93889e-18 6.93889e-18 rpy=3.32777e-18 -2.35601e-17 -9.45252e-18 -> xyz=-6.93889e-18 0 6.93889e-18 rpy=-3.78524e-31 4.09793e-17 2.87272e-31
- joint passive_2_z: origin xyz=0 6.93889e-18 6.93889e-18 rpy=3.32777e-18 -2.35601e-17 -9.45252e-18 -> xyz=-6.93889e-18 0 6.93889e-18 rpy=-3.78524e-31 4.09793e-17 2.87272e-31
- joint passive_3_x: origin xyz=0.0229319 -0.0327739 0.007 rpy=0.365063 0.0882156 -2.70538 -> xyz=0.04 8.32667e-17 0.007 rpy=0.373569 0.0882156 -1.0381
- joint passive_3_y: origin xyz=0 0 0 rpy=-2.43112e-17 2.25632e-17 2.00133e-17 -> xyz=6.93889e-18 0 -1.38778e-17 rpy=4.65239e-19 -4.2966e-17 1.0182e-17
- joint passive_3_z: origin xyz=0 0 0 rpy=-2.43112e-17 2.25632e-17 2.00133e-17 -> xyz=6.93889e-18 0 -1.38778e-17 rpy=4.65239e-19 -4.2966e-17 1.0182e-17
- joint passive_4_x: origin xyz=0.0229319 0.0327739 0.007 rpy=-0.077578 0.0882156 2.70538 -> xyz=0.04 1.38778e-17 0.007 rpy=-0.0860846 0.0882156 1.0381
- joint passive_4_y: origin xyz=1.38778e-17 0 0 rpy=3.17368e-18 -3.23103e-18 -2.7013e-17 -> xyz=1.38778e-17 0 0 rpy=2.88217e-18 2.28461e-18 -8.3094e-17
- joint passive_4_z: origin xyz=1.38778e-17 0 0 rpy=3.17368e-18 -3.23103e-18 -2.7013e-17 -> xyz=1.38778e-17 0 0 rpy=2.88217e-18 2.28461e-18 -8.3094e-17
- joint passive_5_x: origin xyz=0.0229319 -0.0327739 0.007 rpy=0.11547 0.0882156 -2.70538 -> xyz=0.04 6.93889e-17 0.007 rpy=0.123977 0.0882156 -1.0381
- joint passive_5_y: origin xyz=0 0 0 rpy=-3.0015e-19 1.3471e-17 1.28245e-17 -> xyz=-1.38778e-17 -1.38778e-17 6.93889e-18 rpy=-1.54617e-17 2.86037e-17 -1.44876e-17
- joint passive_5_z: origin xyz=0 0 0 rpy=-3.0015e-19 1.3471e-17 1.28245e-17 -> xyz=-1.38778e-17 -1.38778e-17 6.93889e-18 rpy=-1.54617e-17 2.86037e-17 -1.44876e-17
- joint passive_6_x: origin xyz=-0.0327739 0.0229319 0.007 rpy=3.06981 0.0882156 -2.00701 -> xyz=0.04 5.55112e-17 0.007 rpy=3.0613 0.0882156 1.0381
- joint passive_6_y: origin xyz=-2.77556e-17 -1.38778e-17 0 rpy=-2.80507e-17 2.33044e-18 5.49106e-18 -> xyz=6.93889e-18 0 6.93889e-18 rpy=-3.99045e-17 7.78637e-18 -7.13427e-17
- joint passive_6_z: origin xyz=-2.77556e-17 -1.38778e-17 0 rpy=-2.80507e-17 2.33044e-18 5.49106e-18 -> xyz=6.93889e-18 0 6.93889e-18 rpy=-3.99045e-17 7.78637e-18 -7.13427e-17
- joint passive_7_x: origin xyz=-0.085 -1.38778e-17 6.93889e-18 rpy=3.14159 2.33044e-18 5.49106e-18 -> xyz=-0.085 1.38778e-17 6.93889e-18 rpy=3.14159 7.78637e-18 -7.13427e-17
- joint passive_7_y: origin xyz=-2.77556e-17 0 -6.93889e-18 rpy=-2.80507e-17 -2.33044e-18 -5.49106e-18 -> xyz=0 0 0 rpy=-3.99045e-17 -7.78637e-18 7.13427e-17
- joint passive_7_z: origin xyz=-2.77556e-17 0 -6.93889e-18 rpy=-2.80507e-17 -2.33044e-18 -5.49106e-18 -> xyz=0 0 0 rpy=-3.99045e-17 -7.78637e-18 7.13427e-17
- joint right_antenna: origin xyz=-0.0925548 0.0287641 -0.00377325 rpy=1.66493 1.39725 0.631412 -> xyz=-0.0948524 0.0197779 -0.00445785 rpy=1.63922 1.39152 0.701924
- joint stewart_1: origin xyz=-0.0328112 -0.0304906 -0.0418333 rpy=-1.5708 3.05628e-14 -1.0472 -> xyz=-0.0328112 -0.0304906 -0.0418333 rpy=-1.5708 3.50863e-13 -1.0472
- joint stewart_2: origin xyz=-0.0428112 -0.01317 -0.0418333 rpy=-1.5708 6.75017e-15 -1.0472 -> xyz=-0.0428112 -0.01317 -0.0418333 rpy=1.5708 4.23181e-14 2.0944
- joint stewart_3: origin xyz=-0.01 0.0436606 -0.0418333 rpy=1.5708 1.5708 0 -> xyz=-0.01 0.0436606 -0.0418333 rpy=-1.5708 -2.70151e-14 -3.14159
- joint stewart_4: origin xyz=0.01 0.0436606 -0.0418333 rpy=1.5708 1.5708 0 -> xyz=0.01 0.0436606 -0.0418333 rpy=1.5708 -5.41904e-14 -3.32512e-14
- joint stewart_5: origin xyz=0.0428112 -0.01317 -0.0418333 rpy=-2.61799 1.5708 0 -> xyz=0.0428112 -0.01317 -0.0418333 rpy=-1.5708 1.51498e-14 1.0472
- joint stewart_6: origin xyz=0.0328112 -0.0304906 -0.0418333 rpy=-1.5708 1.11952e-14 1.0472 -> xyz=0.0328112 -0.0304906 -0.0418333 rpy=1.5708 2.23981e-14 -2.0944
- joint yaw_body: origin xyz=-2.45997e-07 6.93889e-18 0.0348 rpy=-3.14159 6.78125e-28 -1.5708 -> xyz=-2.45997e-07 6.93889e-18 0.0348 rpy=3.14159 1.34892e-14 -1.5708

File: src/reachy_mini/descriptions/reachy_mini/urdf/robot_no_collision.urdf (robot description, URDF)
Before this commit: robot robot, 45 links, 44 joints
Joints:
- joint camera_frame: origin xyz=-0.0367778 -0.0471665 0.00283045 rpy=1.69996 0.547922 -1.07174 -> xyz=-0.0321159 -0.05047 0.00257878 rpy=1.70724 0.544115 -0.97213
- joint camera_optical_frame: origin xyz=-0.0367778 -0.0471665 0.00283045 rpy=2.93358 1.00937 1.82549 -> xyz=-0.0321159 -0.05047 0.00257878 rpy=2.92045 1.01151 1.9102
- joint closing_1_1_frame: origin xyz=0.085 -1.38778e-17 -6.93889e-18 rpy=-1.89585e-17 -5.12506e-17 5.13924e-17 -> xyz=0.085 -1.38778e-17 -6.93889e-18 rpy=-1.1607e-16 3.42669e-17 4.62147e-17
- joint closing_1_2_frame: origin xyz=0.00583863 -0.022426 0.0368459 rpy=-2.91303 1.06415 -0.938629 -> xyz=0.00768882 -0.0217774 0.0368953 rpy=-2.90143 1.05953 -0.832675
- joint closing_2_1_frame: origin xyz=-0.014684 -0.0833865 -0.00748861 rpy=3.07468 -0.0882156 1.39649 -> xyz=0.043 -0.0729378 -0.00748861 rpy=3.06617 -0.0882156 2.10349
- joint closing_2_2_frame: origin xyz=0.00182437 -0.0169454 0.0490871 rpy=-2.91303 1.06415 -0.938629 -> xyz=0.00307947 -0.0167102 0.049105 rpy=-2.90143 1.05953 -0.832675
- joint closing_3_1_frame: origin xyz=-0.085 -6.93889e-18 0 rpy=-2.43112e-17 2.25632e-17 2.00133e-17 -> xyz=-0.085 0 -1.38778e-17 rpy=4.65239e-19 -4.2966e-17 1.0182e-17
- joint closing_3_2_frame: origin xyz=-0.016495 0.0225206 0.0503005 rpy=-2.93358 -1.00937 -1.3161 -> xyz=-0.0189403 0.0208215 0.050171 rpy=-2.92045 -1.01151 -1.23139
- joint closing_4_1_frame: origin xyz=-0.085 0 0 rpy=3.17368e-18 -3.23103e-18 -2.7013e-17 -> xyz=-0.085 -1.38778e-17 0 rpy=2.88217e-18 2.28461e-18 -8.3094e-17
- joint closing_4_2_frame: origin xyz=-0.0183729 0.0297336 0.0384495 rpy=-2.93358 -1.00937 -1.3161 -> xyz=-0.0214133 0.0278259 0.0383042 rpy=-2.92045 -1.01151 -1.23139
- joint closing_5_1_frame: origin xyz=-0.085 0 0 rpy=-3.0015e-19 1.3471e-17 1.28245e-17 -> xyz=-0.085 -2.77556e-17 1.38778e-17 rpy=-1.54617e-17 2.86037e-17 -1.44876e-17
- joint closing_5_2_frame: origin xyz=-0.00589217 0.0126937 0.00039027 rpy=-3.11354 -0.110171 0.431499 -> xyz=-0.00708235 0.0120716 0.000342873 rpy=-3.11693 -0.116645 0.52771
- joint head_frame: origin xyz=-0.00551617 0.00426275 0.0291789 rpy=1.69996 0.547922 -1.07174 -> xyz=-0.00611127 0.00370522 0.0291364 rpy=1.70724 0.544115 -0.97213
- joint left_antenna: origin xyz=-0.078553 -0.0250168 0.0845885 rpy=2.94387 0.505067 2.01001 -> xyz=-0.0764135 -0.0324475 0.0840224 rpy=2.93649 0.508471 2.10225
- joint passive_1_x: origin xyz=0.0327739 0.0229319 0.007 rpy=-0.129033 -0.0882156 2.00701 -> xyz=0.04 -1.6545e-10 0.007 rpy=-0.13754 -0.0882156 2.10349
- joint passive_1_y: origin xyz=0 0 -6.93889e-18 rpy=-1.89585e-17 -5.12506e-17 5.13924e-17 -> xyz=-1.38778e-17 0 -6.93889e-18 rpy=-1.1607e-16 3.42669e-17 4.62147e-17
- joint passive_1_z: origin xyz=0 0 -6.93889e-18 rpy=-1.89585e-17 -5.12506e-17 5.13924e-17 -> xyz=-1.38778e-17 0 -6.93889e-18 rpy=-1.1607e-16 3.42669e-17 4.62147e-17
- joint passive_2_x: origin xyz=-0.0327739 0.0229319 0.007 rpy=-3.14159 2.27308e-16 -0.610524 -> xyz=0.04 8.32667e-17 0.007 rpy=-3.14159 -9.64904e-17 -3.14159
- joint passive_2_y: origin xyz=0 6.93889e-18 6.93889e-18 rpy=3.32777e-18 -2.35601e-17 -9.45252e-18 -> xyz=-6.93889e-18 0 6.93889e-18 rpy=-3.78524e-31 4.09793e-17 2.87272e-31
- joint passive_2_z: origin xyz=0 6.93889e-18 6.93889e-18 rpy=3.32777e-18 -2.35601e-17 -9.45252e-18 -> xyz=-6.93889e-18 0 6.93889e-18 rpy=-3.78524e-31 4.09793e-17 2.87272e-31
- joint passive_3_x: origin xyz=0.0229319 -0.0327739 0.007 rpy=0.365063 0.0882156 -2.70538 -> xyz=0.04 8.32667e-17 0.007 rpy=0.373569 0.0882156 -1.0381
- joint passive_3_y: origin xyz=0 0 0 rpy=-2.43112e-17 2.25632e-17 2.00133e-17 -> xyz=6.93889e-18 0 -1.38778e-17 rpy=4.65239e-19 -4.2966e-17 1.0182e-17
- joint passive_3_z: origin xyz=0 0 0 rpy=-2.43112e-17 2.25632e-17 2.00133e-17 -> xyz=6.93889e-18 0 -1.38778e-17 rpy=4.65239e-19 -4.2966e-17 1.0182e-17
- joint passive_4_x: origin xyz=0.0229319 0.0327739 0.007 rpy=-0.077578 0.0882156 2.70538 -> xyz=0.04 1.38778e-17 0.007 rpy=-0.0860846 0.0882156 1.0381
- joint passive_4_y: origin xyz=1.38778e-17 0 0 rpy=3.17368e-18 -3.23103e-18 -2.7013e-17 -> xyz=1.38778e-17 0 0 rpy=2.88217e-18 2.28461e-18 -8.3094e-17
- joint passive_4_z: origin xyz=1.38778e-17 0 0 rpy=3.17368e-18 -3.23103e-18 -2.7013e-17 -> xyz=1.38778e-17 0 0 rpy=2.88217e-18 2.28461e-18 -8.3094e-17
- joint passive_5_x: origin xyz=0.0229319 -0.0327739 0.007 rpy=0.11547 0.0882156 -2.70538 -> xyz=0.04 6.93889e-17 0.007 rpy=0.123977 0.0882156 -1.0381
- joint passive_5_y: origin xyz=0 0 0 rpy=-3.0015e-19 1.3471e-17 1.28245e-17 -> xyz=-1.38778e-17 -1.38778e-17 6.93889e-18 rpy=-1.54617e-17 2.86037e-17 -1.44876e-17
- joint passive_5_z: origin xyz=0 0 0 rpy=-3.0015e-19 1.3471e-17 1.28245e-17 -> xyz=-1.38778e-17 -1.38778e-17 6.93889e-18 rpy=-1.54617e-17 2.86037e-17 -1.44876e-17
- joint passive_6_x: origin xyz=-0.0327739 0.0229319 0.007 rpy=3.06981 0.0882156 -2.00701 -> xyz=0.04 5.55112e-17 0.007 rpy=3.0613 0.0882156 1.0381
- joint passive_6_y: origin xyz=-2.77556e-17 -1.38778e-17 0 rpy=-2.80507e-17 2.33044e-18 5.49106e-18 -> xyz=6.93889e-18 0 6.93889e-18 rpy=-3.99045e-17 7.78637e-18 -7.13427e-17
- joint passive_6_z: origin xyz=-2.77556e-17 -1.38778e-17 0 rpy=-2.80507e-17 2.33044e-18 5.49106e-18 -> xyz=6.93889e-18 0 6.93889e-18 rpy=-3.99045e-17 7.78637e-18 -7.13427e-17
- joint passive_7_x: origin xyz=-0.085 -1.38778e-17 6.93889e-18 rpy=3.14159 2.33044e-18 5.49106e-18 -> xyz=-0.085 1.38778e-17 6.93889e-18 rpy=3.14159 7.78637e-18 -7.13427e-17
- joint passive_7_y: origin xyz=-2.77556e-17 0 -6.93889e-18 rpy=-2.80507e-17 -2.33044e-18 -5.49106e-18 -> xyz=0 0 0 rpy=-3.99045e-17 -7.78637e-18 7.13427e-17
- joint passive_7_z: origin xyz=-2.77556e-17 0 -6.93889e-18 rpy=-2.80507e-17 -2.33044e-18 -5.49106e-18 -> xyz=0 0 0 rpy=-3.99045e-17 -7.78637e-18 7.13427e-17
- joint right_antenna: origin xyz=-0.0925548 0.0287641 -0.00377325 rpy=1.66493 1.39725 0.631412 -> xyz=-0.0948524 0.0197779 -0.00445785 rpy=1.63922 1.39152 0.701924
- joint stewart_1: origin xyz=-0.0328112 -0.0304906 -0.0418333 rpy=-1.5708 3.05628e-14 -1.0472 -> xyz=-0.0328112 -0.0304906 -0.0418333 rpy=-1.5708 3.50863e-13 -1.0472
- joint stewart_2: origin xyz=-0.0428112 -0.01317 -0.0418333 rpy=-1.5708 6.75017e-15 -1.0472 -> xyz=-0.0428112 -0.01317 -0.0418333 rpy=1.5708 4.23181e-14 2.0944
- joint stewart_3: origin xyz=-0.01 0.0436606 -0.0418333 rpy=1.5708 1.5708 0 -> xyz=-0.01 0.0436606 -0.0418333 rpy=-1.5708 -2.70151e-14 -3.14159
- joint stewart_4: origin xyz=0.01 0.0436606 -0.0418333 rpy=1.5708 1.5708 0 -> xyz=0.01 0.0436606 -0.0418333 rpy=1.5708 -5.41904e-14 -3.32512e-14
- joint stewart_5: origin xyz=0.0428112 -0.01317 -0.0418333 rpy=-2.61799 1.5708 0 -> xyz=0.0428112 -0.01317 -0.0418333 rpy=-1.5708 1.51498e-14 1.0472
- joint stewart_6: origin xyz=0.0328112 -0.0304906 -0.0418333 rpy=-1.5708 1.11952e-14 1.0472 -> xyz=0.0328112 -0.0304906 -0.0418333 rpy=1.5708 2.23981e-14 -2.0944
- joint yaw_body: origin xyz=-2.45997e-07 6.93889e-18 0.0348 rpy=-3.14159 6.78125e-28 -1.5708 -> xyz=-2.45997e-07 6.93889e-18 0.0348 rpy=3.14159 1.34892e-14 -1.5708
