Commit message: updating urdf and mjcf with actual dof limits

File: src/reachy_mini/descriptions/reachy_mini/urdf/robot.urdf (robot description, URDF)
Before this commit: robot robot, 45 links, 44 joints
Joints:
- joint closing_1_1_frame: origin xyz=0.085 -1.38778e-17 -6.93889e-18 rpy=-1.1607e-16 3.42669e-17 4.62147e-17 -> xyz=0.085 -1.38778e-17 0 rpy=-4.80812e-17 3.69195e-17 -3.11194e-17
- joint closing_3_1_frame: origin xyz=-0.085 0 -1.38778e-17 rpy=4.65239e-19 -4.2966e-17 1.0182e-17 -> xyz=-0.085 -1.38778e-17 0 rpy=-4.71809e-17 -7.61919e-18 5.54539e-17
- joint closing_4_1_frame: origin xyz=-0.085 -1.38778e-17 0 rpy=2.88217e-18 2.28461e-18 -8.3094e-17 -> xyz=-0.085 2.77556e-17 0 rpy=-3.54762e-18 2.76754e-18 -1.40989e-17
- joint closing_5_1_frame: origin xyz=-0.085 -2.77556e-17 1.38778e-17 rpy=-1.54617e-17 2.86037e-17 -1.44876e-17 -> xyz=-0.085 -1.38778e-17 0 rpy=-1.10888e-16 -3.21444e-17 3.55033e-17
- joint passive_1_y: origin xyz=-1.38778e-17 0 -6.93889e-18 rpy=-1.1607e-16 3.42669e-17 4.62147e-17 -> xyz=6.93889e-18 0 0 rpy=-4.80812e-17 3.69195e-17 -3.11194e-17
- joint passive_1_z: origin xyz=-1.38778e-17 0 -6.93889e-18 rpy=-1.1607e-16 3.42669e-17 4.62147e-17 -> xyz=6.93889e-18 0 0 rpy=-4.80812e-17 3.69195e-17 -3.11194e-17
- joint passive_2_x: origin xyz=0.04 8.32667e-17 0.007 rpy=-3.14159 -9.64904e-17 -3.14159 -> xyz=0.04 1.249e-16 0.007 rpy=-3.14159 5.37396e-16 -3.14159
- joint passive_2_y: origin xyz=-6.93889e-18 0 6.93889e-18 rpy=-3.78524e-31 4.09793e-17 2.87272e-31 -> xyz=-6.93889e-18 0 6.93889e-18 rpy=-4.29816e-30 7.32263e-17 -8.42229e-30
- joint passive_2_z: origin xyz=-6.93889e-18 0 6.93889e-18 rpy=-3.78524e-31 4.09793e-17 2.87272e-31 -> xyz=-6.93889e-18 0 6.93889e-18 rpy=-4.29816e-30 7.32263e-17 -8.42229e-30
- joint passive_3_y: origin xyz=6.93889e-18 0 -1.38778e-17 rpy=4.65239e-19 -4.2966e-17 1.0182e-17 -> xyz=-6.93889e-18 0 -1.38778e-17 rpy=-4.71809e-17 -7.61919e-18 5.54539e-17
- joint passive_3_z: origin xyz=6.93889e-18 0 -1.38778e-17 rpy=4.65239e-19 -4.2966e-17 1.0182e-17 -> xyz=-6.93889e-18 0 -1.38778e-17 rpy=-4.71809e-17 -7.61919e-18 5.54539e-17
- joint passive_4_x: origin xyz=0.04 1.38778e-17 0.007 rpy=-0.0860846 0.0882156 1.0381 -> xyz=0.04 2.77556e-17 0.007 rpy=-0.0860846 0.0882156 1.0381
- joint passive_4_y: origin xyz=1.38778e-17 0 0 rpy=2.88217e-18 2.28461e-18 -8.3094e-17 -> xyz=6.93889e-18 0 0 rpy=-3.54762e-18 2.76754e-18 -1.40989e-17
- joint passive_4_z: origin xyz=1.38778e-17 0 0 rpy=2.88217e-18 2.28461e-18 -8.3094e-17 -> xyz=6.93889e-18 0 0 rpy=-3.54762e-18 2.76754e-18 -1.40989e-17
- joint passive_5_x: origin xyz=0.04 6.93889e-17 0.007 rpy=0.123977 0.0882156 -1.0381 -> xyz=0.04 5.55112e-17 0.007 rpy=0.123977 0.0882156 -1.0381
- joint passive_5_y: origin xyz=-1.38778e-17 -1.38778e-17 6.93889e-18 rpy=-1.54617e-17 2.86037e-17 -1.44876e-17 -> xyz=0 0 -6.93889e-18 rpy=-1.10888e-16 -3.21444e-17 3.55033e-17
- joint passive_5_z: origin xyz=-1.38778e-17 -1.38778e-17 6.93889e-18 rpy=-1.54617e-17 2.86037e-17 -1.44876e-17 -> xyz=0 0 -6.93889e-18 rpy=-1.10888e-16 -3.21444e-17 3.55033e-17
- joint passive_6_x: origin xyz=0.04 5.55112e-17 0.007 rpy=3.0613 0.0882156 1.0381 -> xyz=0.04 9.71445e-17 0.007 rpy=3.0613 0.0882156 1.0381
- joint passive_6_y: origin xyz=6.93889e-18 0 6.93889e-18 rpy=-3.99045e-17 7.78637e-18 -7.13427e-17 -> xyz=1.38778e-17 0 0 rpy=-7.27418e-17 2.10388e-17 4.15523e-17
- joint passive_6_z: origin xyz=6.93889e-18 0 6.93889e-18 rpy=-3.99045e-17 7.78637e-18 -7.13427e-17 -> xyz=1.38778e-17 0 0 rpy=-7.27418e-17 2.10388e-17 4.15523e-17
- joint passive_7_x: origin xyz=-0.085 1.38778e-17 6.93889e-18 rpy=3.14159 7.78637e-18 -7.13427e-17 -> xyz=-0.085 0 0 rpy=3.14159 2.10388e-17 4.15523e-17
- joint passive_7_y: origin xyz=0 0 0 rpy=-3.99045e-17 -7.78637e-18 7.13427e-17 -> xyz=0 0 0 rpy=-7.27418e-17 -2.10388e-17 -4.15523e-17
- joint passive_7_z: origin xyz=0 0 0 rpy=-3.99045e-17 -7.78637e-18 7.13427e-17 -> xyz=0 0 0 rpy=-7.27418e-17 -2.10388e-17 -4.15523e-17
- joint stewart_1: limit lower=-3.141592653589793 upper=3.141592653589793 effort=10 velocity=8 -> lower=-0.837758 upper=1.22173 effort=10 velocity=8; origin xyz=-0.0328112 -0.0304906 -0.0418333 rpy=-1.5708 3.50863e-13 -1.0472 -> xyz=-0.0328112 -0.0304906 -0.0418333 rpy=-1.5708 -5.91241e-14 -1.0472
- joint stewart_2: limit lower=-3.141592653589793 upper=3.141592653589793 effort=10 velocity=8 -> lower=-1.22173 upper=1.22173 effort=10 velocity=8; origin xyz=-0.0428112 -0.01317 -0.0418333 rpy=1.5708 4.23181e-14 2.0944 -> xyz=-0.0428112 -0.01317 -0.0418333 rpy=1.5708 -1.47282e-13 2.0944
- joint stewart_3: limit lower=-3.141592653589793 upper=3.141592653589793 effort=10 velocity=8 -> lower=-0.837758 upper=1.22173 effort=10 velocity=8; origin xyz=-0.01 0.0436606 -0.0418333 rpy=-1.5708 -2.70151e-14 -3.14159 -> xyz=-0.01 0.0436606 -0.0418333 rpy=-1.5708 -5.72146e-14 -3.14159
- joint stewart_4: limit lower=-3.141592653589793 upper=3.141592653589793 effort=10 velocity=8 -> lower=-1.22173 upper=0.837758 effort=10 velocity=8; origin xyz=0.01 0.0436606 -0.0418333 rpy=1.5708 -5.41904e-14 -3.32512e-14 -> xyz=0.01 0.0436606 -0.0418333 rpy=1.5708 7.49452e-14 -3.47181e-14
- joint stewart_5: limit lower=-3.141592653589793 upper=3.141592653589793 effort=10 velocity=8 -> lower=-1.22173 upper=1.22173 effort=10 velocity=8; origin xyz=0.0428112 -0.01317 -0.0418333 rpy=-1.5708 1.51498e-14 1.0472 -> xyz=0.0428112 -0.01317 -0.0418333 rpy=-1.5708 1.79054e-13 1.0472
- joint stewart_6: limit lower=-3.141592653589793 upper=3.141592653589793 effort=10 velocity=8 -> lower=-1.22173 upper=0.837758 effort=10 velocity=8; origin xyz=0.0328112 -0.0304906 -0.0418333 rpy=1.5708 2.23981e-14 -2.0944 -> xyz=0.0328112 -0.0304906 -0.0418333 rpy=1.5708 5.32144e-14 -2.0944
- joint yaw_body: origin xyz=-2.45997e-07 6.93889e-18 0.0348 rpy=3.14159 1.34892e-14 -1.5708 -> xyz=-2.45997e-07 6.93889e-18 0.0348 rpy=3.14159 1.77636e-15 -1.5708

File: src/reachy_mini/descriptions/reachy_mini/urdf/robot_no_collision.urdf (robot description, URDF)
Before this commit: robot robot, 45 links, 44 joints
Joints:
- joint closing_1_1_frame: origin xyz=0.085 -1.38778e-17 -6.93889e-18 rpy=-1.1607e-16 3.42669e-17 4.62147e-17 -> xyz=0.085 -1.38778e-17 0 rpy=-4.80812e-17 3.69195e-17 -3.11194e-17
- joint closing_3_1_frame: origin xyz=-0.085 0 -1.38778e-17 rpy=4.65239e-19 -4.2966e-17 1.0182e-17 -> xyz=-0.085 -1.38778e-17 0 rpy=-4.71809e-17 -7.61919e-18 5.54539e-17
- joint closing_4_1_frame: origin xyz=-0.085 -1.38778e-17 0 rpy=2.88217e-18 2.28461e-18 -8.3094e-17 -> xyz=-0.085 2.77556e-17 0 rpy=-3.54762e-18 2.76754e-18 -1.40989e-17
- joint closing_5_1_frame: origin xyz=-0.085 -2.77556e-17 1.38778e-17 rpy=-1.54617e-17 2.86037e-17 -1.44876e-17 -> xyz=-0.085 -1.38778e-17 0 rpy=-1.10888e-16 -3.21444e-17 3.55033e-17
- joint passive_1_y: origin xyz=-1.38778e-17 0 -6.93889e-18 rpy=-1.1607e-16 3.42669e-17 4.62147e-17 -> xyz=6.93889e-18 0 0 rpy=-4.80812e-17 3.69195e-17 -3.11194e-17
- joint passive_1_z: origin xyz=-1.38778e-17 0 -6.93889e-18 rpy=-1.1607e-16 3.42669e-17 4.62147e-17 -> xyz=6.93889e-18 0 0 rpy=-4.80812e-17 3.69195e-17 -3.11194e-17
- joint passive_2_x: origin xyz=0.04 8.32667e-17 0.007 rpy=-3.14159 -9.64904e-17 -3.14159 -> xyz=0.04 1.249e-16 0.007 rpy=-3.14159 5.37396e-16 -3.14159
- joint passive_2_y: origin xyz=-6.93889e-18 0 6.93889e-18 rpy=-3.78524e-31 4.09793e-17 2.87272e-31 -> xyz=-6.93889e-18 0 6.93889e-18 rpy=-4.29816e-30 7.32263e-17 -8.42229e-30
- joint passive_2_z: origin xyz=-6.93889e-18 0 6.93889e-18 rpy=-3.78524e-31 4.09793e-17 2.87272e-31 -> xyz=-6.93889e-18 0 6.93889e-18 rpy=-4.29816e-30 7.32263e-17 -8.42229e-30
- joint passive_3_y: origin xyz=6.93889e-18 0 -1.38778e-17 rpy=4.65239e-19 -4.2966e-17 1.0182e-17 -> xyz=-6.93889e-18 0 -1.38778e-17 rpy=-4.71809e-17 -7.61919e-18 5.54539e-17
- joint passive_3_z: origin xyz=6.93889e-18 0 -1.38778e-17 rpy=4.65239e-19 -4.2966e-17 1.0182e-17 -> xyz=-6.93889e-18 0 -1.38778e-17 rpy=-4.71809e-17 -7.61919e-18 5.54539e-17
- joint passive_4_x: origin xyz=0.04 1.38778e-17 0.007 rpy=-0.0860846 0.0882156 1.0381 -> xyz=0.04 2.77556e-17 0.007 rpy=-0.0860846 0.0882156 1.0381
- joint passive_4_y: origin xyz=1.38778e-17 0 0 rpy=2.88217e-18 2.28461e-18 -8.3094e-17 -> xyz=6.93889e-18 0 0 rpy=-3.54762e-18 2.76754e-18 -1.40989e-17
- joint passive_4_z: origin xyz=1.38778e-17 0 0 rpy=2.88217e-18 2.28461e-18 -8.3094e-17 -> xyz=6.93889e-18 0 0 rpy=-3.54762e-18 2.76754e-18 -1.40989e-17
- joint passive_5_x: origin xyz=0.04 6.93889e-17 0.007 rpy=0.123977 0.0882156 -1.0381 -> xyz=0.04 5.55112e-17 0.007 rpy=0.123977 0.0882156 -1.0381
- joint passive_5_y: origin xyz=-1.38778e-17 -1.38778e-17 6.93889e-18 rpy=-1.54617e-17 2.86037e-17 -1.44876e-17 -> xyz=0 0 -6.93889e-18 rpy=-1.10888e-16 -3.21444e-17 3.55033e-17
- joint passive_5_z: origin xyz=-1.38778e-17 -1.38778e-17 6.93889e-18 rpy=-1.54617e-17 2.86037e-17 -1.44876e-17 -> xyz=0 0 -6.93889e-18 rpy=-1.10888e-16 -3.21444e-17 3.55033e-17
- joint passive_6_x: origin xyz=0.04 5.55112e-17 0.007 rpy=3.0613 0.0882156 1.0381 -> xyz=0.04 9.71445e-17 0.007 rpy=3.0613 0.0882156 1.0381
- joint passive_6_y: origin xyz=6.93889e-18 0 6.93889e-18 rpy=-3.99045e-17 7.78637e-18 -7.13427e-17 -> xyz=1.38778e-17 0 0 rpy=-7.27418e-17 2.10388e-17 4.15523e-17
- joint passive_6_z: origin xyz=6.93889e-18 0 6.93889e-18 rpy=-3.99045e-17 7.78637e-18 -7.13427e-17 -> xyz=1.38778e-17 0 0 rpy=-7.27418e-17 2.10388e-17 4.15523e-17
- joint passive_7_x: origin xyz=-0.085 1.38778e-17 6.93889e-18 rpy=3.14159 7.78637e-18 -7.13427e-17 -> xyz=-0.085 0 0 rpy=3.14159 2.10388e-17 4.15523e-17
- joint passive_7_y: origin xyz=0 0 0 rpy=-3.99045e-17 -7.78637e-18 7.13427e-17 -> xyz=0 0 0 rpy=-7.27418e-17 -2.10388e-17 -4.15523e-17
- joint passive_7_z: origin xyz=0 0 0 rpy=-3.99045e-17 -7.78637e-18 7.13427e-17 -> xyz=0 0 0 rpy=-7.27418e-17 -2.10388e-17 -4.15523e-17
- joint stewart_1: limit lower=-3.141592653589793 upper=3.141592653589793 effort=10 velocity=8 -> lower=-0.837758 upper=1.22173 effort=10 velocity=8; origin xyz=-0.0328112 -0.0304906 -0.0418333 rpy=-1.5708 3.50863e-13 -1.0472 -> xyz=-0.0328112 -0.0304906 -0.0418333 rpy=-1.5708 -5.91241e-14 -1.0472
- joint stewart_2: limit lower=-3.141592653589793 upper=3.141592653589793 effort=10 velocity=8 -> lower=-1.22173 upper=1.22173 effort=10 velocity=8; origin xyz=-0.0428112 -0.01317 -0.0418333 rpy=1.5708 4.23181e-14 2.0944 -> xyz=-0.0428112 -0.01317 -0.0418333 rpy=1.5708 -1.47282e-13 2.0944
- joint stewart_3: limit lower=-3.141592653589793 upper=3.141592653589793 effort=10 velocity=8 -> lower=-0.837758 upper=1.22173 effort=10 velocity=8; origin xyz=-0.01 0.0436606 -0.0418333 rpy=-1.5708 -2.70151e-14 -3.14159 -> xyz=-0.01 0.0436606 -0.0418333 rpy=-1.5708 -5.72146e-14 -3.14159
- joint stewart_4: limit lower=-3.141592653589793 upper=3.141592653589793 effort=10 velocity=8 -> lower=-1.22173 upper=0.837758 effort=10 velocity=8; origin xyz=0.01 0.0436606 -0.0418333 rpy=1.5708 -5.41904e-14 -3.32512e-14 -> xyz=0.01 0.0436606 -0.0418333 rpy=1.5708 7.49452e-14 -3.47181e-14
- joint stewart_5: limit lower=-3.141592653589793 upper=3.141592653589793 effort=10 velocity=8 -> lower=-1.22173 upper=1.22173 effort=10 velocity=8; origin xyz=0.0428112 -0.01317 -0.0418333 rpy=-1.5708 1.51498e-14 1.0472 -> xyz=0.0428112 -0.01317 -0.0418333 rpy=-1.5708 1.79054e-13 1.0472
- joint stewart_6: limit lower=-3.141592653589793 upper=3.141592653589793 effort=10 velocity=8 -> lower=-1.22173 upper=0.837758 effort=10 velocity=8; origin xyz=0.0328112 -0.0304906 -0.0418333 rpy=1.5708 2.23981e-14 -2.0944 -> xyz=0.0328112 -0.0304906 -0.0418333 rpy=1.5708 5.32144e-14 -2.0944
- joint yaw_body: origin xyz=-2.45997e-07 6.93889e-18 0.0348 rpy=3.14159 1.34892e-14 -1.5708 -> xyz=-2.45997e-07 6.93889e-18 0.0348 rpy=3.14159 1.77636e-15 -1.5708

Commit message: change body_yaw direction, update limits. urdf and mjcf are updated

File: src/reachy_mini/descriptions/reachy_mini/urdf/robot.urdf (robot description, URDF)
Before this commit: robot robot, 45 links, 44 joints
Joints:
- joint dummy_yaw: origin xyz=0 0 0 rpy=3.14 0 -1.57 -> xyz=0 0 0 rpy=3.14 0 1.57
- joint stewart_1: limit lower=-0.837758 upper=1.22173 effort=10 velocity=8 -> lower=-0.837758 upper=1.39626 effort=10 velocity=8; origin xyz=-0.0328112 -0.0304906 -0.0418333 rpy=-1.5708 -5.91241e-14 -1.0472 -> xyz=-0.0328112 0.0304906 0.0418333 rpy=1.5708 5.91241e-14 1.0472
- joint stewart_2: limit lower=-1.22173 upper=1.22173 effort=10 velocity=8 -> lower=-1.39626 upper=1.22173 effort=10 velocity=8; origin xyz=-0.0428112 -0.01317 -0.0418333 rpy=1.5708 -1.47282e-13 2.0944 -> xyz=-0.0428112 0.01317 0.0418333 rpy=-1.5708 1.47282e-13 -2.0944
- joint stewart_3: limit lower=-0.837758 upper=1.22173 effort=10 velocity=8 -> lower=-0.837758 upper=1.39626 effort=10 velocity=8; origin xyz=-0.01 0.0436606 -0.0418333 rpy=-1.5708 -5.72146e-14 -3.14159 -> xyz=-0.01 -0.0436606 0.0418333 rpy=1.5708 5.72146e-14 3.14159
- joint stewart_4: limit lower=-1.22173 upper=0.837758 effort=10 velocity=8 -> lower=-1.39626 upper=0.837758 effort=10 velocity=8; origin xyz=0.01 0.0436606 -0.0418333 rpy=1.5708 7.49452e-14 -3.47181e-14 -> xyz=0.01 -0.0436606 0.0418333 rpy=-1.5708 -7.49452e-14 3.47181e-14
- joint stewart_5: limit lower=-1.22173 upper=1.22173 effort=10 velocity=8 -> lower=-1.22173 upper=1.39626 effort=10 velocity=8; origin xyz=0.0428112 -0.01317 -0.0418333 rpy=-1.5708 1.79054e-13 1.0472 -> xyz=0.0428112 0.01317 0.0418333 rpy=1.5708 -1.79054e-13 -1.0472
- joint stewart_6: limit lower=-1.22173 upper=0.837758 effort=10 velocity=8 -> lower=-1.39626 upper=0.837758 effort=10 velocity=8; origin xyz=0.0328112 -0.0304906 -0.0418333 rpy=1.5708 5.32144e-14 -2.0944 -> xyz=0.0328112 0.0304906 0.0418333 rpy=-1.5708 -5.32144e-14 2.0944
- joint yaw_body: limit lower=-3.141592653589793 upper=3.141592653589793 effort=10 velocity=8 -> lower=-2.79253 upper=2.79253 effort=10 velocity=8; origin xyz=-2.45997e-07 6.93889e-18 0.0348 rpy=3.14159 1.77636e-15 -1.5708 -> xyz=-2.45997e-07 6.93889e-18 0.0348 rpy=-3.74039e-16 1.77636e-15 -1.5708

File: src/reachy_mini/descriptions/reachy_mini/urdf/robot_no_collision.urdf (robot description, URDF)
Before this commit: robot robot, 45 links, 44 joints
Joints:
- joint dummy_yaw: origin xyz=0 0 0 rpy=3.14 0 -1.57 -> xyz=0 0 0 rpy=3.14 0 1.57
- joint stewart_1: limit lower=-0.837758 upper=1.22173 effort=10 velocity=8 -> lower=-0.837758 upper=1.39626 effort=10 velocity=8; origin xyz=-0.0328112 -0.0304906 -0.0418333 rpy=-1.5708 -5.91241e-14 -1.0472 -> xyz=-0.0328112 0.0304906 0.0418333 rpy=1.5708 5.91241e-14 1.0472
- joint stewart_2: limit lower=-1.22173 upper=1.22173 effort=10 velocity=8 -> lower=-1.39626 upper=1.22173 effort=10 velocity=8; origin xyz=-0.0428112 -0.01317 -0.0418333 rpy=1.5708 -1.47282e-13 2.0944 -> xyz=-0.0428112 0.01317 0.0418333 rpy=-1.5708 1.47282e-13 -2.0944
- joint stewart_3: limit lower=-0.837758 upper=1.22173 effort=10 velocity=8 -> lower=-0.837758 upper=1.39626 effort=10 velocity=8; origin xyz=-0.01 0.0436606 -0.0418333 rpy=-1.5708 -5.72146e-14 -3.14159 -> xyz=-0.01 -0.0436606 0.0418333 rpy=1.5708 5.72146e-14 3.14159
- joint stewart_4: limit lower=-1.22173 upper=0.837758 effort=10 velocity=8 -> lower=-1.39626 upper=0.837758 effort=10 velocity=8; origin xyz=0.01 0.0436606 -0.0418333 rpy=1.5708 7.49452e-14 -3.47181e-14 -> xyz=0.01 -0.0436606 0.0418333 rpy=-1.5708 -7.49452e-14 3.47181e-14
- joint stewart_5: limit lower=-1.22173 upper=1.22173 effort=10 velocity=8 -> lower=-1.22173 upper=1.39626 effort=10 velocity=8; origin xyz=0.0428112 -0.01317 -0.0418333 rpy=-1.5708 1.79054e-13 1.0472 -> xyz=0.0428112 0.01317 0.0418333 rpy=1.5708 -1.79054e-13 -1.0472
- joint stewart_6: limit lower=-1.22173 upper=0.837758 effort=10 velocity=8 -> lower=-1.39626 upper=0.837758 effort=10 velocity=8; origin xyz=0.0328112 -0.0304906 -0.0418333 rpy=1.5708 5.32144e-14 -2.0944 -> xyz=0.0328112 0.0304906 0.0418333 rpy=-1.5708 -5.32144e-14 2.0944
- joint yaw_body: limit lower=-3.141592653589793 upper=3.141592653589793 effort=10 velocity=8 -> lower=-2.79253 upper=2.79253 effort=10 velocity=8; origin xyz=-2.45997e-07 6.93889e-18 0.0348 rpy=3.14159 1.77636e-15 -1.5708 -> xyz=-2.45997e-07 6.93889e-18 0.0348 rpy=-3.74039e-16 1.77636e-15 -1.5708
